File: amr_stm32_kicad/amr_stm32_kicad.kicad_pcb (KiCad board)
At the start: 2 copper layers, 21 parts, among them U1 LMR33640ADDA, U2 SGM2205-3.3

Commit message: update1
Parts:
- added C13: 22uF/10V, Capacitor_SMD:C_0805_2012Metric, F.Cu at (106.9, 13.0)
- added C14: 100nF/50V, Capacitor_SMD:C_0805_2012Metric, F.Cu at (106.9, 16.0)
- added C15: 100nF/50V, Capacitor_SMD:C_0805_2012Metric, F.Cu at (106.9, 19.0)
- added C16: 1uF/16V, Capacitor_SMD:C_0805_2012Metric, F.Cu at (106.9, 22.0)
- added C17: 100nF/50V, Capacitor_SMD:C_0805_2012Metric, F.Cu at (106.9, 25.0)
- added D4: TVS_Diode 5.0V, Diode_SMD:D_SMB, F.Cu at (108.9, 29.3)
- added F1: PTC Fuse 3A, Fuse:Fuse_1812_4532Metric, F.Cu at (108.1, 34.6)
- added J1: Header 2x20, Connector_PinHeader_2.54mm:PinHeader_2x20_P2.54mm_Vertical, F.Cu at (96.5, 13.5)
- added R4: 10kOhm, Resistor_SMD:R_0805_2012Metric, F.Cu at (106.8, 42.6)
- added U3: BMI323, BMI323:BMI323_BOS, F.Cu at (107.0, 39.1)

Commit message: update2
Parts:
- added C18: 10uF/25V, Capacitor_SMD:CP_Elec_6.3x7.7, F.Cu at (95.6, -2.88)
- added C19: 100nF/50V, Capacitor_SMD:C_0805_2012Metric, F.Cu at (73.7, -31.0)
- added C20: 100nF/50V, Capacitor_SMD:C_0805_2012Metric, F.Cu at (73.7, -28.0)
- added C21: 20pF/50V, Capacitor_SMD:C_0805_2012Metric, F.Cu at (73.7, -25.0)
- added C22: 20pF/50V, Capacitor_SMD:C_0805_2012Metric, F.Cu at (73.7, -22.0)
- added C23: 20pF/50V, Capacitor_SMD:C_0805_2012Metric, F.Cu at (73.7, -19.0)
- added C24: 20pF/50V, Capacitor_SMD:C_0805_2012Metric, F.Cu at (73.7, -15.9)
- added C25: 100nF, Capacitor_SMD:C_0603_1608Metric, F.Cu at (69.5, -31.2)
- added C26: 100nF, Capacitor_SMD:C_0603_1608Metric, F.Cu at (69.5, -28.7)
- added C27: 100nF, Capacitor_SMD:C_0603_1608Metric, F.Cu at (69.5, -26.2)
- added C28: 100nF, Capacitor_SMD:C_0603_1608Metric, F.Cu at (69.5, -23.7)
- added C29: 100nF, Capacitor_SMD:C_0603_1608Metric, F.Cu at (69.5, -21.2)
- added C30: 1uF, Capacitor_SMD:C_0603_1608Metric, F.Cu at (69.5, -18.7)
- added C31: 100nF, Capacitor_SMD:C_0603_1608Metric, F.Cu at (69.5, -16.2)
- added C32: 2.2uF, Capacitor_SMD:C_0603_1608Metric, F.Cu at (69.5, -13.7)
- added C33: 2.2uF, Capacitor_SMD:C_0603_1608Metric, F.Cu at (69.5, -11.2)
- added FB1: FerriteBead, Inductor_SMD:L_0805_2012Metric, F.Cu at (78.2, -1.07)
- added J2: MA, Connector_JST:JST_XH_B6B-XH-A_1x06_P2.50mm_Vertical, F.Cu at (79.4, -29.1)
- added J3: MB, Connector_JST:JST_XH_B6B-XH-A_1x06_P2.50mm_Vertical, F.Cu at (79.4, -21.3)
- added R10: 10kOhm, Resistor_SMD:R_0805_2012Metric, F.Cu at (97.6, -19.2)
- added R5: 10kOhm, Resistor_SMD:R_0805_2012Metric, F.Cu at (97.6, -31.0)
- added R7: 10kOhm, Resistor_SMD:R_0805_2012Metric, F.Cu at (97.6, -28.1)
- added R8: 10kOhm, Resistor_SMD:R_0805_2012Metric, F.Cu at (97.6, -25.1)
- added R9: 10kOhm, Resistor_SMD:R_0805_2012Metric, F.Cu at (97.6, -22.2)
- added U4: TB6612FNG, Package_SO:SSOP-24_5.3x8.2mm_P0.65mm, F.Cu at (95.6, -11.8)
- added U5: STM32F405RGTx, Package_QFP:LQFP-64_10x10mm_P0.5mm, F.Cu at (83.2, -9.68)

Commit message: update3
Parts:
- added C34: 22pF, Capacitor_SMD:C_0603_1608Metric, F.Cu at (114.5, -16.7)
- added C35: 22pF, Capacitor_SMD:C_0603_1608Metric, F.Cu at (114.5, -14.2)
- added C36: 100nF, Capacitor_SMD:C_0603_1608Metric, F.Cu at (114.5, -11.7)
- added C37: 100nF, Capacitor_SMD:C_0603_1608Metric, F.Cu at (114.5, -9.21)
- added R11: 10kOhm, Resistor_SMD:R_0603_1608Metric, F.Cu at (114.5, -4.20)
- added R6: 10kOhm, Resistor_SMD:R_0603_1608Metric, F.Cu at (114.5, -6.71)
- added SW1: SW_Reset, Button_Switch_SMD:SW_SPST_B3U-1000P, F.Cu at (119.4, -15.8)
- added SW2: SW_BOOT, Button_Switch_SMD:SW_SPST_B3U-1000P, F.Cu at (119.4, -11.5)
- added Y1: 8MHz, Crystal:Crystal_SMD_5032-2Pin_5.0x3.2mm, F.Cu at (120.2, -6.67)
Connections:
- U5 pad 46: unconnected-(U5-PA13-Pad46) -> /STM32_SWDIO
- U5 pad 49: unconnected-(U5-PA14-Pad49) -> /STM32_SWCLK
- U5 pad 5: unconnected-(U5-PH0-Pad5) -> Net-(U5-PH0)
- U5 pad 6: unconnected-(U5-PH1-Pad6) -> Net-(U5-PH1)
- U5 pad 60: unconnected-(U5-BOOT0-Pad60) -> /STM32_BOOT
- U5 pad 7: unconnected-(U5-NRST-Pad7) -> /STM32_RESET

Commit message: update4
Parts:
- added C38: 470nF, Capacitor_SMD:C_0603_1608Metric, F.Cu at (69.2, 66.3)
- added C39: 100nF, Capacitor_SMD:C_0603_1608Metric, F.Cu at (69.2, 68.8)
- added J4: ST_Link, Connector_PinHeader_2.54mm:PinHeader_2x04_P2.54mm_Horizontal, F.Cu at (69.5, 79.8)
- added J5: USB_C_Receptacle_USB2.0_16P, Connector_USB:USB_C_Receptacle_HRO_TYPE-C-31-M-12, F.Cu at (61.3, 70.8)
- added J6: USB_C_Receptacle_USB2.0_16P, Connector_USB:USB_C_Receptacle_HRO_TYPE-C-31-M-12, F.Cu at (61.3, 81.3)
- added Q1: Q_PMOS_GSD, Package_TO_SOT_SMD:SOT-23, F.Cu at (76.9, 92.0)
- added R12: 5.1kOhm, Resistor_SMD:R_0603_1608Metric, F.Cu at (69.2, 71.3)
- added R13: 5.1kOhm, Resistor_SMD:R_0603_1608Metric, F.Cu at (69.2, 73.8)
- added R14: 10kOhm, Resistor_SMD:R_0603_1608Metric, F.Cu at (69.2, 76.3)
- added R15: 2kOhm, Resistor_SMD:R_0603_1608Metric, F.Cu at (73.2, 66.3)
- added R16: 9kOhm, Resistor_SMD:R_0603_1608Metric, F.Cu at (73.2, 68.8)
- added R17: 1kOhm, Resistor_SMD:R_0603_1608Metric, F.Cu at (73.2, 71.3)
- added R18: 470Ohm, Resistor_SMD:R_0603_1608Metric, F.Cu at (73.2, 73.8)
- added R19: 470Ohm, Resistor_SMD:R_0603_1608Metric, F.Cu at (73.2, 76.3)
- added R20: 470Ohm, Resistor_SMD:R_0603_1608Metric, F.Cu at (77.2, 66.3)
- added R21: 5.1kOhm, Resistor_SMD:R_0603_1608Metric, F.Cu at (77.2, 68.8)
- added R22: 5.1kOhm, Resistor_SMD:R_0603_1608Metric, F.Cu at (77.2, 71.3)
- added U6: LM358, Package_SO:SOIC-8_3.9x4.9mm_P1.27mm, F.Cu at (59.7, 89.3)
- added U7: CH340E, Package_SO:MSOP-10_3x3mm_P0.5mm, F.Cu at (70.8, 92.1)
Connections:
- C1 pad 1: +12V -> VCC
- C2 pad 1: +12V -> VCC
- C8 pad 1: +12V -> VCC
- U1 pad 2: +12V -> VCC
- U1 pad 3: +12V -> VCC
- U5 pad 14: unconnected-(U5-PA0-Pad14) -> /RX_USB
- U5 pad 15: unconnected-(U5-PA1-Pad15) -> /TX_USB
- U5 pad 44: unconnected-(U5-PA11-Pad44) -> /USB_DM
- U5 pad 45: unconnected-(U5-PA12-Pad45) -> /USB_DP
- U5 pad 54: unconnected-(U5-PD2-Pad54) -> /IMU_CS
- U5 pad 55: unconnected-(U5-PB3-Pad55) -> /IMU_SCK
- U5 pad 56: unconnected-(U5-PB4-Pad56) -> /IMU_MISO
- U5 pad 57: unconnected-(U5-PB5-Pad57) -> /IMU_MOSI
- U5 pad 61: unconnected-(U5-PB8-Pad61) -> /IMU_INT

Commit message: update5
Parts:
- added D5: LED_RUN, LED_SMD:LED_0603_1608Metric, F.Cu at (114.1, 51.3)
- added D6: LED_ERR, LED_SMD:LED_0603_1608Metric, F.Cu at (114.1, 53.9)
- added J7: +12V_BAT, Connector_AMASS:AMASS_XT60PW-M_1x02_P7.20mm_Horizontal, F.Cu at (99.7, 67.4)
- added R23: 330 Ohm, Resistor_SMD:R_0603_1608Metric, F.Cu at (114.1, 56.4)
- added R24: 330 Ohm, Resistor_SMD:R_0603_1608Metric, F.Cu at (114.1, 58.9)
- moved J2 152.1 mm to (156.5, 102.0)
- moved J6 139.0 mm to (200.0, 90.5), turned to 90 degrees
- moved J5 138.9 mm to (200.0, 63.0), turned to 90 degrees
- moved J3 135.5 mm to (135.5, 102.0)
- moved U5 122.7 mm to (171.0, 76.0)
- moved J4 121.7 mm to (191.0, 73.0)
- moved J1 51.8 mm to (127.5, 55.0), turned to 90 degrees
- moved C34 11.4 mm to (125.7, -15.0)
- moved C35 11.4 mm to (125.7, -12.5)
- moved C36 11.4 mm to (125.7, -10.0)
- moved C37 11.4 mm to (125.7, -7.50)
- moved R11 11.4 mm to (125.7, -2.48)
- moved R6 11.4 mm to (125.7, -4.99)
- moved SW1 11.4 mm to (130.7, -14.1)
- moved SW2 11.4 mm to (130.7, -9.76)
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Connections:
- C1 pad 1: VCC -> /+12V_BAT
- C18 pad 1: +12V -> /+12V_BAT
- C19 pad 1: +12V -> /+12V_BAT
- C2 pad 1: VCC -> /+12V_BAT
- C8 pad 1: VCC -> /+12V_BAT
- J1 pad 14: unconnected-(J1-Pin_14-Pad14) -> GND
- J1 pad 2: unconnected-(J1-Pin_2-Pad2) -> /+5V_Pi
- J1 pad 20: unconnected-(J1-Pin_20-Pad20) -> GND
- J1 pad 25: unconnected-(J1-Pin_25-Pad25) -> GND
- J1 pad 3: unconnected-(J1-Pin_3-Pad3) -> /SDA_Pi
- J1 pad 30: unconnected-(J1-Pin_30-Pad30) -> GND
- J1 pad 34: unconnected-(J1-Pin_34-Pad34) -> GND
- J1 pad 39: unconnected-(J1-Pin_39-Pad39) -> GND
- J1 pad 4: unconnected-(J1-Pin_4-Pad4) -> /+5V_Pi
- J1 pad 5: unconnected-(J1-Pin_5-Pad5) -> /SCL_Pi
- J1 pad 6: unconnected-(J1-Pin_6-Pad6) -> GND
- J1 pad 9: unconnected-(J1-Pin_9-Pad9) -> GND
- R16 pad 1: VCC -> /+12V_BAT
- U1 pad 2: VCC -> /+12V_BAT
- U1 pad 3: VCC -> /+12V_BAT
- U4 pad 13: +12V -> /+12V_BAT
- U4 pad 14: +12V -> /+12V_BAT
- U4 pad 24: +12V -> /+12V_BAT
- U5 pad 10: unconnected-(U5-PC2-Pad10) -> /STM32_BIN1
- U5 pad 11: unconnected-(U5-PC3-Pad11) -> /STM32_BIN2
- U5 pad 14: /RX_USB -> /ENC_1A
- U5 pad 15: /TX_USB -> /ENC_1B
- U5 pad 21: unconnected-(U5-PA5-Pad21) -> /%BAT
- U5 pad 22: unconnected-(U5-PA6-Pad22) -> /ENC_2A
- U5 pad 23: unconnected-(U5-PA7-Pad23) -> /ENC_2B
- U5 pad 27: unconnected-(U5-PB1-Pad27) -> /LED_RUN
- U5 pad 28: unconnected-(U5-PB2-Pad28) -> /LED_ERR
- U5 pad 39: unconnected-(U5-PC8-Pad39) -> /STM32_PWMA
- U5 pad 40: unconnected-(U5-PC9-Pad40) -> /STM32_PWMB
- U5 pad 42: unconnected-(U5-PA9-Pad42) -> /RX_USB
- U5 pad 43: unconnected-(U5-PA10-Pad43) -> /TX_USB
- U5 pad 58: unconnected-(U5-PB6-Pad58) -> /SCL_Pi
- U5 pad 59: unconnected-(U5-PB7-Pad59) -> /SDA_Pi
- U5 pad 8: unconnected-(U5-PC0-Pad8) -> /STM32_AIN1
- U5 pad 9: unconnected-(U5-PC1-Pad9) -> /STM32_AIN2
Other:
- board outline added: 85 x 56 mm

Commit message: update6
Parts:
- removed C1: 10uF/35V, Capacitor_SMD:C_1206_3216Metric
- removed C2: 220nF/50V, Capacitor_SMD:C_0603_1608Metric
- removed C3: 1uF/16V, Capacitor_SMD:C_0603_1608Metric
- removed C4: 0.1uF/25V, Capacitor_SMD:C_0603_1608Metric
- removed C5, C6, C7: 22uF/16V, Capacitor_SMD:C_0805_2012Metric
- removed C8: 1000uF/35V, Capacitor_THT:CP_Radial_D10.0mm_P5.00mm
- removed L1: 6.8uH/4.5A, Inductor_SMD:L_7.3x7.3_H4.5
- removed R1: 100kOhm, Resistor_SMD:R_0603_1608Metric
- removed R2: 24.9kOhm, Resistor_SMD:R_0603_1608Metric
- removed U1: LMR33640ADDA, Package_SO:Texas_HSOP-8-1EP_3.9x4.9mm_P1.27mm_ThermalVias
- added C40: 10uF, Capacitor_SMD:C_1206_3216Metric, F.Cu at (80.8, 40.7)
- added C41: 0.1uF, Capacitor_SMD:C_0603_1608Metric, F.Cu at (76.0, 28.8)
- added C42: 5pF, Capacitor_SMD:C_0603_1608Metric, F.Cu at (76.0, 31.3)
- added C43: 0.47uF, Capacitor_SMD:C_0603_1608Metric, F.Cu at (76.0, 33.8)
- added C44: 0.1uF, Capacitor_SMD:C_0603_1608Metric, F.Cu at (76.0, 36.3)
- added C45: 22uF, Capacitor_SMD:C_1206_3216Metric, F.Cu at (80.8, 44.1)
- added C46: 22uF, Capacitor_SMD:C_1206_3216Metric, F.Cu at (80.8, 47.4)
- added C47: 10uF, Capacitor_SMD:C_1206_3216Metric, F.Cu at (80.8, 50.8)
- added C48: 1000uF/35V, Capacitor_THT:CP_Radial_D10.0mm_P5.00mm, F.Cu at (81.5, 33.3)
- added L2: 3.3uH, Inductor_SMD:L_7.3x7.3_H4.5, F.Cu at (88.4, 43.5)
- added R25: 374kOhm, Resistor_SMD:R_0603_1608Metric, F.Cu at (76.0, 38.8)
- added R26: 49.9kOhm, Resistor_SMD:R_0603_1608Metric, F.Cu at (76.0, 41.3)
- added R27: 10kOhm, Resistor_SMD:R_0603_1608Metric, F.Cu at (76.0, 43.8)
- added R28: 100kOhm, Resistor_SMD:R_0603_1608Metric, F.Cu at (76.0, 46.3)
- added U9: TPS56528DDA, Package_SO:Texas_HSOP-8-1EP_3.9x4.9mm_P1.27mm_ThermalVias, F.Cu at (94.1, 30.9)
- F1: value PTC Fuse 3A -> Fuse 2920L500; footprint Fuse:Fuse_1812_4532Metric -> Fuse:Fuse_2920_7451Metric
- J2, J3: footprint Connector_JST:JST_XH_B6B-XH-A_1x06_P2.50mm_Vertical -> Connector_JST:JST_PH_S6B-PH-K_1x06_P2.00mm_Horizontal
- moved C25 150.0 mm to (215.2, 6.69)
- moved C26 150.0 mm to (215.2, 9.20)
- moved C27 150.0 mm to (215.2, 11.7)
- moved C28 150.0 mm to (215.2, 14.2)
- moved C29 150.0 mm to (215.2, 16.7)
- moved C30 150.0 mm to (215.2, 19.2)
- moved C31 150.0 mm to (215.2, 21.8)
- moved FB1 150.0 mm to (223.9, 36.9)
- moved C16 86.5 mm to (171.5, 79.5)
- moved C15 86.0 mm to (168.0, 79.5), turned to 180 degrees
- moved C17 79.1 mm to (167.0, 76.5), turned to -90 degrees
- moved U3 73.3 mm to (170.0, 76.5), turned to -90 degrees
- moved R4 70.3 mm to (170.0, 73.5)
- moved C36 59.0 mm to (174.3, 23.5)
- moved R11 59.0 mm to (174.3, 31.0)
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
Commit message: update7
Parts:
- removed D4: TVS_Diode 5.0V, Diode_SMD:D_SMB
- added C1: 2.2uF, Capacitor_SMD:C_0603_1608Metric, F.Cu at (194.0, 54.0)
- added C2: 2.2uF, Capacitor_SMD:C_0603_1608Metric, F.Cu at (196.5, 54.0)
- added D7: SMAJ5.0A, Diode_SMD:D_SMA, F.Cu at (160.5, 61.0)
- added FB2: F120R, Inductor_SMD:L_0603_1608Metric, F.Cu at (199.0, 54.0)
- C13: value 22uF/10V -> 100uF; footprint Capacitor_SMD:C_0805_2012Metric -> Capacitor_Tantalum_SMD:CP_EIA-6032-28_Kemet-C
- Q1: value Q_PMOS_GSD -> FDN304P
- moved C10 144.7 mm to (161.8, 93.6)
- moved C11 144.7 mm to (161.8, 96.7)
- moved C12 144.7 mm to (161.8, 99.7)
- moved C9 144.7 mm to (161.8, 90.6)
- moved D1 144.7 mm to (169.5, 93.0)
- moved D3 144.7 mm to (166.3, 101.7)
- moved R3 144.7 mm to (161.8, 102.6)
- moved U2 144.7 mm to (172.4, 99.3)
- moved D2 144.7 mm to (166.9, 98.5)
- moved C19 141.3 mm to (139.0, 96.5), turned to 90 degrees
- moved C32 140.8 mm to (187.0, 66.0)
- moved C33 140.8 mm to (187.0, 68.5)
- moved C20 140.1 mm to (142.0, 96.5), turned to 90 degrees
- moved C21 139.0 mm to (145.0, 96.5), turned to 90 degrees
- moved C22 138.0 mm to (148.0, 96.5), turned to 90 degrees
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Connections:
- J1 pad 10: unconnected-(J1-Pin_10-Pad10) -> /USART2_TX
- J1 pad 11: unconnected-(J1-Pin_11-Pad11) -> /STM32_RESET
- J1 pad 13: unconnected-(J1-Pin_13-Pad13) -> /STM32_BOOT
- J1 pad 8: unconnected-(J1-Pin_8-Pad8) -> /USART2_RX
- Q1 pad 3: +5V -> Net-(Q1-D)
- U5 pad 16: unconnected-(U5-PA2-Pad16) -> /USART2_TX
- U5 pad 17: unconnected-(U5-PA3-Pad17) -> /USART2_RX

Commit message: update8
Parts:
- removed C13: 100uF, Capacitor_Tantalum_SMD:CP_EIA-6032-28_Kemet-C
- removed C14: 100nF/50V, Capacitor_SMD:C_0805_2012Metric
- removed D7: SMAJ5.0A, Diode_SMD:D_SMA
- removed F1: Fuse 2920L500, Fuse:Fuse_2920_7451Metric
- added J8: USB_A, Connector_USB:USB_A_Molex_67643_Horizontal, F.Cu at (164.0, 94.1)
- moved R3 21.7 mm to (163.0, 81.0), turned to 90 degrees
- moved D2 20.0 mm to (151.5, 85.9), turned to 90 degrees
- moved D3 19.0 mm to (155.0, 86.4)
- moved C12 18.8 mm to (160.0, 81.0), turned to 90 degrees
- moved U2 18.2 mm to (159.0, 86.9)
- moved C11 16.4 mm to (157.0, 81.0), turned to 90 degrees
- moved C10 14.9 mm to (154.0, 81.0), turned to 90 degrees
- moved C9 14.5 mm to (151.0, 81.0), turned to 90 degrees
- moved R16 11.9 mm to (154.2, 69.0)
- moved R17 11.9 mm to (154.2, 66.5)
- moved C38 11.9 mm to (154.4, 60.0)
- moved R18 11.9 mm to (154.2, 64.0)
- moved U6 11.9 mm to (160.5, 61.5)
- moved D1 6.95 mm to (166.0, 87.0)
- moved C15 5.15 mm to (162.5, 75.5)
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Connections:
- J1 pad 2: /+5V_Pi -> unconnected-(J1-Pin_2-Pad2)
- J1 pad 4: /+5V_Pi -> unconnected-(J1-Pin_4-Pad4)
