File: amr_stm32_kicad/amr_stm32_kicad.kicad_pcb (KiCad board)
At the start: 4 copper layers, 85 x 56 mm, 96 parts, among them J1 Header 2x20, J10 VCC, J2 Motor_Left, J3 Motor_right, J4 ST_Link, J5 USB_FS_Interface, J6 USB_UART, J7 +12V_BAT, J8 USB_A_Pi, J9 UART, Q1 FDN304P, SW1 SW_Reset, SW2 SW_BOOT, U2 SGM2205-3.3, U3 BMI323, U4 TB6612FNG, U5 STM32F405RGTx, U6 LM358, U7 CH340E, U9 TPS56528DDA, Y2 8MHz

Commit message: update14
Parts:
- U3: footprint BMI323:BMI323_BOS -> BMI323:BMI323_BOS-L
- moved R4 1.18 mm to (162.0, 61.2), turned to -90 degrees
- moved J7 0.50 mm to (136.2, 69.1)
- moved C15 0.41 mm to (166.3, 58.5)
- moved C16 0.41 mm to (162.8, 58.5)
- moved C33 0.35 mm to (175.0, 63.8)
Routing:
- net +5V: track 212.8 -> 221.2 mm
- net GND: track 28.0 -> 33.4 mm, vias 108 -> 89
- net Net-(Q1-G): track 26.0 -> 30.3 mm
- net /IMU_INT: track 9.45 -> 12.5 mm
- net /IMU_SCK: track 7.52 -> 9.62 mm
- net Net-(D3-A): track 0.00 -> 2.01 mm
- net /ENC_1A: track 41.0 -> 39.3 mm
- net /USART2_RX: track 51.2 -> 52.7 mm, vias 6 -> 4
- net /+3.3VA: track 8.33 -> 6.83 mm
- net /USB_DM: track 40.5 -> 42.0 mm
- net /ENC_1B: track 40.8 -> 42.2 mm
- net Net-(U5-PH0): track 29.9 -> 31.2 mm
- net /LED_RUN: track 11.9 -> 13.1 mm
- net VBUS: track 58.0 -> 59.2 mm
- net /LED_ERR: track 9.36 -> 10.6 mm
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- removed copper zone on B.Cu, net GND

Commit message: update16
Parts:
- moved Y2 21.7 mm to (162.6, 76.8), turned to 135 degrees
- moved C34 19.9 mm to (163.9, 73.3), turned to 135 degrees
- moved C35 15.4 mm to (166.1, 75.4), turned to -45 degrees
- moved R24 12.0 mm to (182.1, 84.2), turned to 180 degrees
- moved R3 11.8 mm to (158.2, 71.2)
- moved D3 11.7 mm to (156.2, 71.2)
- moved R23 11.4 mm to (182.1, 82.7), turned to 180 degrees
- moved FB1 10.3 mm to (173.8, 80.2), turned to 90 degrees
- moved D6 10.1 mm to (179.1, 84.2), turned to 0 degrees
- moved D5 10.1 mm to (179.0, 82.7), turned to 0 degrees
- moved C30 9.66 mm to (172.0, 80.1), turned to -90 degrees
- moved C31 9.33 mm to (170.5, 80.1), turned to -90 degrees
- moved C25 9.10 mm to (181.8, 60.0), turned to 0 degrees
- moved C27 7.46 mm to (163.8, 70.8), turned to 180 degrees
- moved U5 6.83 mm to (174.5, 69.8)
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Routing:
- net Net-(U5-PH0): track 31.2 -> 10.4 mm, vias 4 -> 0
- net GND: track 33.4 -> 52.4 mm, vias 89 -> 79
- net Net-(U5-PH1): track 26.4 -> 7.70 mm, vias 2 -> 0
- net +3.3V: track 70.6 -> 89.1 mm, vias 40 -> 32
- net +5V: track 221.2 -> 207.0 mm, vias 37 -> 28
- net /STM32_SWDIO: track 44.4 -> 33.4 mm
- net /%BAT: track 13.0 -> 23.9 mm, vias 2 -> 0
- net /USART3_RX: track 36.1 -> 28.4 mm
- net /STM32_BIN1: track 24.4 -> 31.8 mm
- net /ENC_1A: track 39.3 -> 46.5 mm, vias 3 -> 5
- net /USART3_TX: track 33.6 -> 26.5 mm, vias 2 -> 0
- net /ENC_1B: track 42.2 -> 48.9 mm
- net /IMU_SCK: track 9.62 -> 16.2 mm
- net /STM32_BIN2: track 24.8 -> 30.9 mm
- net /RX_USB: track 14.8 -> 9.17 mm
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- added copper zone on B.Cu, net GND

Commit message: update15
Other:
- board text added: "design: @hongtannnn"

Commit message: update18
Parts:
- renumbered SW2 to BOOT, SW1 to RESET
Routing:
- net /ENC_1B: track 48.9 -> 40.1 mm
- net /J1_MA+: track 17.2 -> 23.2 mm
- net /+12V_BAT: track 25.7 -> 20.1 mm
- net GND: track 52.4 -> 48.0 mm
- net /ENC_2A: track 37.0 -> 40.6 mm
- net /ENC_2B: track 34.0 -> 36.0 mm
- net Net-(Q1-G): track 30.3 -> 31.6 mm
- net /ENC_1A: track 46.5 -> 45.3 mm, vias 5 -> 4
- net /J2_MB+: track 26.6 -> 25.4 mm
- net Net-(U5-PH0): track 10.4 -> 11.2 mm
Other:
- board text added: "amr"

Commit message: update19
Parts:
- removed BOOT: SW_BOOT, Button_Switch_SMD:SW_SPST_B3U-1000P
- removed RESET: SW_Reset, Button_Switch_SMD:SW_SPST_B3U-1000P
- added SW1: SW_Reset, Button_Switch_SMD:SW_SPST_B3U-1000P, F.Cu at (192.2, 76.0)
- added SW2: SW_BOOT, Button_Switch_SMD:SW_SPST_B3U-1000P, F.Cu at (192.2, 79.8)
- moved C25 1.25 mm to (181.8, 58.8)
- moved C33 1.25 mm to (181.5, 60.5)
- moved R19 1.06 mm to (184.8, 66.0), turned to 180 degrees
- moved R20 1.06 mm to (184.8, 64.5), turned to 0 degrees
Connections:
- U5 pad 24: /PC4 -> /LED_RUN
- U5 pad 25: /PC5 -> /LED_ERR
- U5 pad 27: /LED_RUN -> /PB1
- U5 pad 28: /LED_ERR -> /PB2
Routing:
- net +3.3V: track 89.1 -> 100.2 mm, vias 32 -> 30
- net /IMU_INT: track 13.2 -> 16.9 mm
- net /IMU_SCK: track 16.2 -> 12.7 mm
- net /USART2_RX: track 55.4 -> 58.9 mm
- net /STM32_RESET: track 71.7 -> 75.1 mm
- net /USART2_TX: track 52.0 -> 55.2 mm
- net GND: track 48.0 -> 44.9 mm, vias 79 -> 77
- net /USB_DP: track 41.3 -> 44.3 mm
- net /STM32_BOOT: track 77.3 -> 74.4 mm
- net /USB_DM: track 41.4 -> 44.0 mm, vias 4 -> 2
- net /TX_USB: track 9.25 -> 6.72 mm
- net /RX_USB: track 9.17 -> 6.76 mm
- net /STM32_PWMA: track 46.6 -> 48.5 mm
- net /STM32_SWDIO: track 33.4 -> 34.7 mm
- net /STM32_PWMB: track 41.2 -> 42.3 mm
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- removed copper zone on F.Cu, net /STM32_RESET

Commit message: update20
Parts:
- added D7: LED_ERR, LED_SMD:LED_0603_1608Metric, F.Cu at (179.0, 85.8)
- added R29: 330 Ohm, Resistor_SMD:R_0603_1608Metric, F.Cu at (182.1, 85.8)
- added REF**: MountingHole_2.7mm_M2.5_DIN965_Pad, MountingHole:MountingHole_2.7mm_M2.5_DIN965_Pad, F.Cu at (122.8, 102.5)
- added REF**: MountingHole_2.7mm_M2.5_DIN965_Pad, MountingHole:MountingHole_2.7mm_M2.5_DIN965_Pad, F.Cu at (180.8, 53.5)
- added REF**: MountingHole_2.7mm_M2.5_DIN965_Pad, MountingHole:MountingHole_2.7mm_M2.5_DIN965_Pad, F.Cu at (122.8, 53.5)
- added REF**: MountingHole_2.7mm_M2.5_DIN965_Pad, MountingHole:MountingHole_2.7mm_M2.5_DIN965_Pad, F.Cu at (180.8, 102.5)
Connections:
- net /LED_ERR renamed /LED_2
- net /LED_RUN renamed /LED_1
- U5 pad 26: /PB0 -> /LED_3
- U5 pad 53: /PC12 -> /IMU_INT
- U5 pad 61: /IMU_INT -> /PB8
Routing:
- net /LED_3: track 0.00 -> 15.1 mm
- net /IMU_INT: track 16.9 -> 8.51 mm
- net +3.3V: track 100.2 -> 103.0 mm, vias 30 -> 29
- net Net-(U5-VCAP_1): track 4.21 -> 5.65 mm
- net Net-(D7-A): track 0.00 -> 1.42 mm
- net /STM32_PWMA: track 48.5 -> 49.5 mm
- net /J1_MA+: track 23.2 -> 22.4 mm
- net /J2_MB+: track 25.4 -> 26.2 mm
- net /USART3_RX: track 28.4 -> 29.0 mm

Commit message: update_photo
Parts:
- renumbered SW2 to BOOT, SW1 to RESET
Changed lines of the file:
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@@
 		(descr "Ultra-small-sized Tactile Switch with High Contact Reliability, Top-actuated Model, without Ground Terminal, without Boss")
 		(tags "Tactile Switch")
-		(property "Reference" "SW1"
+		(property "Reference" "RESET"
 			(at 0 -2.5 0)
 			(layer "F.SilkS")
@@
 			(layer "F.Fab")
 		)
-		(fp_text user "${REFERENCE}"
-			(at 0 -2.5 0)
-			(layer "F.Fab")
-			(effects
-				(font
-					(size 1 1)
-					(thickness 0.15)
-				)
-			)
-		)
 		(pad "1" smd rect
 			(at -1.7 0)
@@
 		(descr "Ultra-small-sized Tactile Switch with High Contact Reliability, Top-actuated Model, without Ground Terminal, without Boss")
 		(tags "Tactile Switch")
-		(property "Reference" "SW2"
-			(at 0 -2.5 0)
+		(property "Reference" "BOOT"
+			(at -0.175 2.475 0)
 			(layer "F.SilkS")
 			(effects
@@
 			(layer "F.Fab")
 		)
-		(fp_text user "${REFERENCE}"
-			(at 0 -2.5 0)
-			(layer "F.Fab")
-			(effects
-				(font
-					(size 1 1)
-					(thickness 0.15)
-				)
-			)
-		)
 		(pad "1" smd rect
 			(at -1.7 0)
@@
 	)
 	(segment
+		(start 180.818198 78.431802)
+		(end 180.818198 75.714644)
+		(width 0.25)
+		(layer "F.Cu")
+		(net "/LED_2")
+	)
+	(segment
+		(start 182.912646 84.25)
+		(end 183.637645 83.525001)
+		(width 0.25)
+		(layer "F.Cu")
+		(net "/LED_2")
+	)
+	(segment
+		(start 183.637645 81.251249)
+		(end 180.818198 78.431802)
+		(width 0.25)
+		(layer "F.Cu")
+		(net "/LED_2")
+	)
+	(segment
+		(start 183.637645 83.525001)
+		(end 183.637645 81.251249)
+		(width 0.25)
+		(layer "F.Cu")
+		(net "/LED_2")
+	)
+	(segment
+		(start 180.818198 75.714644)
+		(end 178.689608 73.586054)
+		(width 0.25)
+		(layer "F.Cu")
+		(net "/LED_2")
+	)
+	(segment
 		(start 179.848433 84.25)
 		(end 181.262646 84.25)
@@
 	)
 	(segment
+		(start 179.8325 85.75)
+		(end 181.25 85.75)
+		(width 0.25)
+		(layer "F.Cu")
+		(net "Net-(D7-A)")
+	)
+	(segment
 		(start 176.214734 63.439072)
 		(end 179.153806 60.5)
@@
 	)
 	(segment
+		(start 184.087645 80.837645)
+		(end 181.268198 78.018198)
+		(width 0.25)
+		(layer "F.Cu")
+		(net "/LED_3")
+	)
+	(segment
+		(start 182.9 85.75)
+		(end 184.087645 84.562355)
+		(width 0.25)
+		(layer "F.Cu")
+		(net "/LED_3")
+	)
+	(segment
+		(start 181.268198 78.018198)
+		(end 181.268198 75.457538)
+		(width 0.25)
+		(layer "F.Cu")
+		(net "/LED_3")
+	)
+	(segment
+		(start 181.268198 75.457538)
+		(end 179.043161 73.232501)
+		(width 0.25)
+		(layer "F.Cu")
+		(net "/LED_3")
+	)
+	(segment
+		(start 184.087645 84.562355)
+		(end 184.087645 80.837645)
+		(width 0.25)
+		(layer "F.Cu")
+		(net "/LED_3")
+	)
+	(segment
+		(start 182.912645 82.744497)
+		(end 182.912645 81.162645)
+		(width 0.25)
+		(layer "F.Cu")
+		(net "/LED_1")
+	)
+	(segment
+		(start 180.25 75.853554)
+		(end 178.336054 73.939608)
+		(width 0.25)
+		(layer "F.Cu")
+		(net "/LED_1")
+	)
+	(segment
+		(start 180.25 78.5)
+		(end 180.25 75.853554)
+		(width 0.25)
+		(layer "F.Cu")
+		(net "/LED_1")
+	)
+	(segment
+		(start 182.912645 81.162645)
+		(end 180.25 78.5)
+		(width 0.25)
+		(layer "F.Cu")
+		(net "/LED_1")
+	)
+	(segment
 		(start 193.75 90.5)
 		(end 194.5 91.25)
@@
 		(net "Net-(J5-CC1)")
 	)
-	(segment
-		(start 179.8325 85.75)
-		(end 181.25 85.75)
-		(width 0.25)
-		(layer "F.Cu")
-		(net "Net-(D7-A)")
-	)
-	(segment
-		(start 182.912645 82.744497)
-		(end 182.912645 81.162645)
-		(width 0.25)
-		(layer "F.Cu")
-		(net "/LED_1")
-	)
-	(segment
-		(start 180.25 75.853554)
-		(end 178.336054 73.939608)
-		(width 0.25)
-		(layer "F.Cu")
-		(net "/LED_1")
-	)
-	(segment
-		(start 180.25 78.5)
-		(end 180.25 75.853554)
-		(width 0.25)
-		(layer "F.Cu")
-		(net "/LED_1")
-	)
-	(segment
-		(start 182.912645 81.162645)
-		(end 180.25 78.5)
-		(width 0.25)
-		(layer "F.Cu")
-		(net "/LED_1")
-	)
-	(segment
-		(start 180.818198 78.431802)
-		(end 180.818198 75.714644)
-		(width 0.25)
-		(layer "F.Cu")
-		(net "/LED_2")
-	)
-	(segment
-		(start 182.912646 84.25)
-		(end 183.637645 83.525001)
-		(width 0.25)
-		(layer "F.Cu")
-		(net "/LED_2")
-	)
-	(segment
-		(start 183.637645 81.251249)
-		(end 180.818198 78.431802)
-		(width 0.25)
-		(layer "F.Cu")
-		(net "/LED_2")
-	)
-	(segment
-		(start 183.637645 83.525001)
-		(end 183.637645 81.251249)
-		(width 0.25)
-		(layer "F.Cu")
-		(net "/LED_2")
-	)
-	(segment
-		(start 180.818198 75.714644)
-		(end 178.689608 73.586054)
-		(width 0.25)
-		(layer "F.Cu")
-		(net "/LED_2")
-	)
-	(segment
-		(start 184.087645 80.837645)
-		(end 181.268198 78.018198)
-		(width 0.25)
-		(layer "F.Cu")
-		(net "/LED_3")
-	)
-	(segment
-		(start 182.9 85.75)
-		(end 184.087645 84.562355)
-		(width 0.25)
-		(layer "F.Cu")
-		(net "/LED_3")
-	)
-	(segment
-		(start 181.268198 78.018198)
-		(end 181.268198 75.457538)
-		(width 0.25)
-		(layer "F.Cu")
-		(net "/LED_3")
-	)
-	(segment
-		(start 181.268198 75.457538)
-		(end 179.043161 73.232501)
-		(width 0.25)
-		(layer "F.Cu")
-		(net "/LED_3")
-	)
-	(segment
-		(start 184.087645 84.562355)
-		(end 184.087645 80.837645)
-		(width 0.25)
-		(layer "F.Cu")
-		(net "/LED_3")
-	)
 	(zone

Commit message: update21
Parts:
- moved C15 3.55 mm to (162.8, 58.5), turned to 180 degrees
- moved C16 3.50 mm to (166.2, 58.5), turned to 0 degrees
- moved R21 0.50 mm to (193.2, 68.5)
Routing:
- net VBUS: track 59.2 -> 73.3 mm
- net +3.3V: track 103.0 -> 109.5 mm, vias 29 -> 26
- net GND: track 45.2 -> 40.0 mm
- net /ENC_1A: track 45.3 -> 41.3 mm
- net /VBAT_SNS: track 5.48 -> 8.49 mm
- net Net-(U6A--): track 0.00 -> 2.82 mm
- net Net-(D1-K): track 16.5 -> 18.7 mm
- net /UART_DP: track 6.52 -> 8.56 mm
- net /J2_MB+: track 26.2 -> 25.4 mm
