File: amr_stm32_kicad/amr_stm32_kicad.kicad_pcb (KiCad board)
At the start: 4 copper layers, 85 x 56 mm, 102 parts, among them J1 Header 2x20, J10 VCC, J2 Motor_Left, J3 Motor_right, J4 ST_Link, J5 USB_FS_Interface, J6 USB_UART, J7 +12V_BAT, J8 USB_A_Pi, J9 UART, Q1 FDN304P, U2 SGM2205-3.3, U3 BMI323, U4 TB6612FNG, U5 STM32F405RGTx, U6 LM358, U7 CH340E, U9 TPS56528DDA, Y2 8MHz

Commit message: update22
Routing:
- net GND: vias 77 -> 143
- net /+12V_BAT: vias 30 -> 27

Commit message: update23
Parts:
- removed REF** (x4): MountingHole_2.7mm_M2.5_DIN965_Pad, MountingHole:MountingHole_2.7mm_M2.5_DIN965_Pad
- moved BOOT 0.08 mm to (192.2, 79.8)
Connections:
- J1 pad 11: /STM32_RESET -> unconnected-(J1-Pin_11-Pad11)
- J1 pad 13: /STM32_BOOT -> unconnected-(J1-Pin_13-Pad13)
Routing:
- net /STM32_RESET: track 75.1 -> 35.3 mm, vias 1 -> 0
- net /STM32_BOOT: track 74.4 -> 41.0 mm, vias 4 -> 2
- net /USART2_RX: track 58.9 -> 61.0 mm
- net /USART2_TX: track 55.2 -> 57.2 mm
- net Net-(U5-VCAP_1): track 5.65 -> 4.22 mm
- net /SDA_Pi: track 47.3 -> 48.1 mm
- net /SCL_Pi: track 44.8 -> 45.5 mm
- net +3.3V: track 109.5 -> 109.0 mm

Commit message: update24
Other:
- board text added: "design by @hongtannnn"
- board text removed: "design: @hongtannnn"
Changed lines of the file:
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@@
 		)
 	)
-	(gr_text "design: @hongtannnn"
+	(gr_text "design by @hongtannnn"
 		(at 181 98 0)
 		(layer "F.SilkS")
@@
 	)
 	(segment
+		(start 171.780241 69.5)
+		(end 170.573654 68.293413)
+		(width 0.2)
+		(layer "F.Cu")
+		(net "/STM32_BOOT")
+	)
+	(segment
+		(start 193.95 79.75)
+		(end 193.95 81.55)
+		(width 0.3)
+		(layer "F.Cu")
+		(net "/STM32_BOOT")
+	)
+	(segment
+		(start 187.325 80.25)
+		(end 187.25 80.325)
+		(width 0.5)
+		(layer "F.Cu")
+		(net "/STM32_BOOT")
+	)
+	(segment
+		(start 187.25 80.325)
+		(end 186.075 80.325)
+		(width 0.25)
+		(layer "F.Cu")
+		(net "/STM32_BOOT")
+	)
+	(segment
+		(start 188.675 80.325)
+		(end 188.75 80.25)
+		(width 0.3)
+		(layer "F.Cu")
+		(net "/STM32_BOOT")
+	)
+	(segment
+		(start 189.5 82.75)
+		(end 188.75 82)
+		(width 0.3)
+		(layer "F.Cu")
+		(net "/STM32_BOOT")
+	)
+	(segment
+		(start 192.75 82.75)
+		(end 189.5 82.75)
+		(width 0.3)
+		(layer "F.Cu")
+		(net "/STM32_BOOT")
+	)
+	(segment
+		(start 185.25 75)
+		(end 186 74.25)
+		(width 0.25)
+		(layer "F.Cu")
+		(net "/STM32_BOOT")
+	)
+	(segment
+		(start 193.95 81.55)
+		(end 192.75 82.75)
+		(width 0.3)
+		(layer "F.Cu")
+		(net "/STM32_BOOT")
+	)
+	(segment
+		(start 187.25 80.325)
+		(end 188.675 80.325)
+		(width 0.3)
+		(layer "F.Cu")
+		(net "/STM32_BOOT")
+	)
+	(segment
+		(start 186.075 80.325)
+		(end 185.25 79.5)
+		(width 0.25)
+		(layer "F.Cu")
+		(net "/STM32_BOOT")
+	)
+	(segment
+		(start 188.75 82)
+		(end 188.75 80.25)
+		(width 0.3)
+		(layer "F.Cu")
+		(net "/STM32_BOOT")
+	)
+	(segment
+		(start 185.25 79.5)
+		(end 185.25 75)
+		(width 0.25)
+		(layer "F.Cu")
+		(net "/STM32_BOOT")
+	)
+	(segment
+		(start 186 74.25)
+		(end 186 73.5)
+		(width 0.25)
+		(layer "F.Cu")
+		(net "/STM32_BOOT")
+	)
+	(segment
+		(start 182.53033 70.03033)
+		(end 175.5 70.03033)
+		(width 0.25)
+		(layer "F.Cu")
+		(net "/STM32_BOOT")
+	)
+	(segment
+		(start 169.254847 66.974606)
+		(end 169.249732 66.974606)
+		(width 0.2)
+		(layer "F.Cu")
+		(net "/STM32_BOOT")
+	)
+	(segment
+		(start 170.206587 67.926346)
+		(end 169.254847 66.974606)
+		(width 0.2)
+		(layer "F.Cu")
+		(net "/STM32_BOOT")
+	)
+	(segment
+		(start 175.5 70.03033)
+		(end 175.5 70.075)
+		(width 0.25)
+		(layer "F.Cu")
+		(net "/STM32_BOOT")
+	)
+	(segment
+		(start 186 73.5)
+		(end 182.53033 70.03033)
+		(width 0.25)
+		(layer "F.Cu")
+		(net "/STM32_BOOT")
+	)
+	(segment
+		(start 170.75 68.474874)
+		(end 169.249732 66.974606)
+		(width 0.2)
+		(layer "F.Cu")
+		(net "/STM32_BOOT")
+	)
+	(via
+		(at 175.5 70.075)
+		(size 0.5)
+		(drill 0.3)
+		(layers "F.Cu" "B.Cu")
+		(net "/STM32_BOOT")
+	)
+	(via
+		(at 171.780241 69.5)
+		(size 0.5)
+		(drill 0.3)
+		(layers "F.Cu" "B.Cu")
+		(net "/STM32_BOOT")
+	)
+	(segment
+		(start 171.780241 69.5)
+		(end 172.355241 70.075)
+		(width 0.25)
+		(layer "B.Cu")
+		(net "/STM32_BOOT")
+	)
+	(segment
+		(start 172.355241 70.075)
+		(end 175.5 70.075)
+		(width 0.25)
+		(layer "B.Cu")
+		(net "/STM32_BOOT")
+	)
+	(segment
 		(start 162.1875 92.0299)
 		(end 161.6576 91.5)
@@
 	)
 	(segment
-		(start 171.780241 69.5)
-		(end 170.573654 68.293413)
-		(width 0.2)
-		(layer "F.Cu")
-		(net "/STM32_BOOT")
-	)
-	(segment
-		(start 193.95 79.75)
-		(end 193.95 81.55)
-		(width 0.3)
-		(layer "F.Cu")
-		(net "/STM32_BOOT")
-	)
-	(segment
-		(start 187.325 80.25)
-		(end 187.25 80.325)
-		(width 0.5)
-		(layer "F.Cu")
-		(net "/STM32_BOOT")
-	)
-	(segment
-		(start 187.25 80.325)
-		(end 186.075 80.325)
-		(width 0.25)
-		(layer "F.Cu")
-		(net "/STM32_BOOT")
-	)
-	(segment
-		(start 188.675 80.325)
-		(end 188.75 80.25)
-		(width 0.3)
-		(layer "F.Cu")
-		(net "/STM32_BOOT")
-	)
-	(segment
-		(start 189.5 82.75)
-		(end 188.75 82)
-		(width 0.3)
-		(layer "F.Cu")
-		(net "/STM32_BOOT")
-	)
-	(segment
-		(start 192.75 82.75)
-		(end 189.5 82.75)
-		(width 0.3)
-		(layer "F.Cu")
-		(net "/STM32_BOOT")
-	)
-	(segment
-		(start 185.25 75)
-		(end 186 74.25)
-		(width 0.25)
-		(layer "F.Cu")
-		(net "/STM32_BOOT")
-	)
-	(segment
-		(start 193.95 81.55)
-		(end 192.75 82.75)
-		(width 0.3)
-		(layer "F.Cu")
-		(net "/STM32_BOOT")
-	)
-	(segment
-		(start 187.25 80.325)
-		(end 188.675 80.325)
-		(width 0.3)
-		(layer "F.Cu")
-		(net "/STM32_BOOT")
-	)
-	(segment
-		(start 186.075 80.325)
-		(end 185.25 79.5)
-		(width 0.25)
-		(layer "F.Cu")
-		(net "/STM32_BOOT")
-	)
-	(segment
-		(start 188.75 82)
-		(end 188.75 80.25)
-		(width 0.3)
-		(layer "F.Cu")
-		(net "/STM32_BOOT")
-	)
-	(segment
-		(start 185.25 79.5)
-		(end 185.25 75)
-		(width 0.25)
-		(layer "F.Cu")
-		(net "/STM32_BOOT")
-	)
-	(segment
-		(start 186 74.25)
-		(end 186 73.5)
-		(width 0.25)
-		(layer "F.Cu")
-		(net "/STM32_BOOT")
-	)
-	(segment
-		(start 182.53033 70.03033)
-		(end 175.5 70.03033)
-		(width 0.25)
-		(layer "F.Cu")
-		(net "/STM32_BOOT")
-	)
-	(segment
-		(start 169.254847 66.974606)
-		(end 169.249732 66.974606)
-		(width 0.2)
-		(layer "F.Cu")
-		(net "/STM32_BOOT")
-	)
-	(segment
-		(start 170.206587 67.926346)
-		(end 169.254847 66.974606)
-		(width 0.2)
-		(layer "F.Cu")
-		(net "/STM32_BOOT")
-	)
-	(segment
-		(start 175.5 70.03033)
-		(end 175.5 70.075)
-		(width 0.25)
-		(layer "F.Cu")
-		(net "/STM32_BOOT")
-	)
-	(segment
-		(start 186 73.5)
-		(end 182.53033 70.03033)
-		(width 0.25)
-		(layer "F.Cu")
-		(net "/STM32_BOOT")
-	)
-	(segment
-		(start 170.75 68.474874)
-		(end 169.249732 66.974606)
-		(width 0.2)
-		(layer "F.Cu")
-		(net "/STM32_BOOT")
-	)
-	(via
-		(at 175.5 70.075)
-		(size 0.5)
-		(drill 0.3)
-		(layers "F.Cu" "B.Cu")
-		(net "/STM32_BOOT")
-	)
-	(via
-		(at 171.780241 69.5)
-		(size 0.5)
-		(drill 0.3)
-		(layers "F.Cu" "B.Cu")
-		(net "/STM32_BOOT")
-	)
-	(segment
-		(start 171.780241 69.5)
-		(end 172.355241 70.075)
-		(width 0.25)
-		(layer "B.Cu")
-		(net "/STM32_BOOT")
-	)
-	(segment
-		(start 172.355241 70.075)
-		(end 175.5 70.075)
-		(width 0.25)
-		(layer "B.Cu")
-		(net "/STM32_BOOT")
-	)
-	(segment

Commit message: update25
Parts:
- moved C45 0.50 mm to (142.9, 62.5)
- moved C46 0.50 mm to (140.5, 62.5)
- moved C10 0.40 mm to (145.8, 63.0)
- moved C9 0.40 mm to (147.8, 63.0)
- moved R11 0.35 mm to (189.0, 76.3)
- moved J4 0.32 mm to (197.1, 73.9)
- moved C36 0.25 mm to (189.0, 79.5)
- moved C37 0.22 mm to (187.2, 76.2)
Routing:
- net +5V: track 207.0 -> 208.9 mm, vias 28 -> 27
- net GND: track 40.0 -> 38.2 mm, vias 143 -> 142
- net /STM32_BOOT: track 41.0 -> 39.6 mm
- net Net-(D1-K): track 18.7 -> 17.7 mm
- net /UART_DM: track 7.99 -> 7.09 mm
- net /ENC_1A: vias 4 -> 3

Commit message: update26
Parts:
- added REF**: MountingHole_2.7mm_M2.5_DIN965_Pad, MountingHole:MountingHole_2.7mm_M2.5_DIN965_Pad, F.Cu at (122.8, 102.5)
- added REF**: MountingHole_2.7mm_M2.5_DIN965_Pad, MountingHole:MountingHole_2.7mm_M2.5_DIN965_Pad, F.Cu at (180.8, 102.5)
- added REF**: MountingHole_2.7mm_M2.5_DIN965_Pad, MountingHole:MountingHole_2.7mm_M2.5_DIN965_Pad, F.Cu at (180.8, 53.5)
- added REF**: MountingHole_2.7mm_M2.5_DIN965_Pad, MountingHole:MountingHole_2.7mm_M2.5_DIN965_Pad, F.Cu at (122.8, 53.5)
- moved C10 2.25 mm to (148.0, 63.0)
- moved C9 2.01 mm to (145.8, 63.0)
- moved C19 0.56 mm to (153.0, 84.0), turned to 180 degrees
Routing:
- net GND: track 38.2 -> 34.0 mm, vias 142 -> 140
- net +5V: track 208.9 -> 207.3 mm
- net Net-(D1-K): track 17.7 -> 16.7 mm
- net +3.3V: track 108.8 -> 108.4 mm, vias 26 -> 27
- net /+12V_BAT: vias 27 -> 22
Other:
- board text added: "+3.3V"
- board text added: "+5V"
- board text added: "GND"
- board text added: "Motor Left"
- board text added: "Motor Right"
- board text added: "RESET"
- board text added: "RX"
- board text added: "SWCLK"
- board text added: "SWDIO"
- board text added: "TX"
- board text added: "USB Full Speed"
- board text added: "USB Pi Power"
- board text added: "USB UART"
- board text added: "VBUS"
- board text added: "designed by @hongtannnn"
- board text removed: "design by @hongtannnn"

Commit message: update28
Parts:
- removed REF** (x4): MountingHole_2.7mm_M2.5_DIN965_Pad, MountingHole:MountingHole_2.7mm_M2.5_DIN965_Pad
- moved C10 3.87 mm to (149.8, 59.5), turned to 90 degrees
- moved C9 2.47 mm to (147.8, 61.5)
- moved D2 2.25 mm to (145.5, 60.5), turned to -90 degrees
- moved C45 2.03 mm to (143.0, 60.5), turned to 90 degrees
- moved C46 2.00 mm to (140.5, 60.5), turned to 90 degrees
- moved D1 0.85 mm to (153.2, 59.2)
- moved C11 0.50 mm to (156.0, 63.0)
- moved C12 0.50 mm to (158.0, 63.0)
- moved U2 0.45 mm to (152.0, 63.0)
Routing:
- net Net-(D1-K): track 16.7 -> 9.74 mm
- net +5V: track 207.3 -> 211.1 mm, vias 27 -> 13
- net GND: track 34.0 -> 32.0 mm, vias 140 -> 135
- net +3.3V: track 108.4 -> 108.9 mm, vias 27 -> 29
- net /+12V_BAT: vias 22 -> 18
- added copper zone on F.Cu, net Net-(D1-K)
