File: amr_stm32_kicad/amr_stm32_kicad.kicad_sch (KiCad schematic)
At the start: 21 parts, among them U1 LMR33640ADDA, U2 SGM2205-3.3

Commit message: update1
Parts:
- added C13: 22uF/10V, Capacitor_SMD:C_0805_2012Metric, symbol Device:C
- added C14, C15, C17: 100nF/50V, Capacitor_SMD:C_0805_2012Metric, symbol Device:C
- added C16: 1uF/16V, Capacitor_SMD:C_0805_2012Metric, symbol Device:C
- added D4: TVS_Diode 5.0V, Diode_SMD:D_SMB, symbol Device:D_TVS
- added F1: PTC Fuse 3A, Fuse:Fuse_1812_4532Metric, symbol Device:Polyfuse_Small
- added J1: Header 2x20, Connector_PinHeader_2.54mm:PinHeader_2x20_P2.54mm_Vertical, symbol Connector_Generic:Conn_02x20_Odd_Even
- added R4: 10kOhm, Resistor_SMD:R_0805_2012Metric, symbol Device:R
- added U3: BMI323, BMI323_BOS, symbol BMI323:BMI323
Connections:
- net +3.3V: now also C15.1, C16.1, C17.1, R4.1, U3.5 (VDDIO), U3.8 (VDD)
- net +5V: now also F1.1
- net GND: now also C13.2, C14.2, C15.2, C16.2, C17.2, D4.1 (A1), U3.6 (GNDIO), U3.7 (GND)
- new net +5V_Pi: C13.1, C14.1, D4.2 (A2), F1.2
- new net IMU_CS: R4.2, U3.12 (CSB)
- new net IMU_INT: U3.4 (INT1)
- new net IMU_MISO: U3.1 (SDO)
- new net IMU_MOSI: U3.14 (SDX)
- new net IMU_SCK: U3.13 (SCX)
- no-connect marks 0 -> 1
Other:
- note added: "IMU SENSOR"
- note added: "POWER PROTECTION Pi"

Commit message: update2
Parts:
- added C18: 10uF/25V, Capacitor_SMD:CP_Elec_6.3x7.7, symbol Device:C_Polarized
- added C19, C20: 100nF/50V, Capacitor_SMD:C_0805_2012Metric, symbol Device:C
- added C21, C22, C23, C24: 20pF/50V, Capacitor_SMD:C_0805_2012Metric, symbol Device:C
- added C25, C26, C27, C28, C29, C31: 100nF, Capacitor_SMD:C_0603_1608Metric, symbol Device:C
- added C30: 1uF, Capacitor_SMD:C_0603_1608Metric, symbol Device:C
- added C32, C33: 2.2uF, Capacitor_SMD:C_0603_1608Metric, symbol Device:C
- added FB1: FerriteBead, Inductor_SMD:L_0805_2012Metric, symbol Device:FerriteBead
- added J2: MA, Connector_JST:JST_XH_B6B-XH-A_1x06_P2.50mm_Vertical, symbol Connector_Generic:Conn_01x06
- added J3: MB, Connector_JST:JST_XH_B6B-XH-A_1x06_P2.50mm_Vertical, symbol Connector_Generic:Conn_01x06
- added R10, R5, R7, R8, R9: 10kOhm, Resistor_SMD:R_0805_2012Metric, symbol Device:R
- added U4: TB6612FNG, Package_SO:SSOP-24_5.3x8.2mm_P0.65mm, symbol Driver_Motor:TB6612FNG
- added U5: STM32F405RGTx, Package_QFP:LQFP-64_10x10mm_P0.5mm, symbol MCU_ST_STM32F4:STM32F405RGTx
Connections:
- net +12V: now also C18.1, C19.1, U4.13 (VM2), U4.14 (VM3), U4.24 (VM1)
- net +3.3V: now also C20.1, C25.1, C26.1, C27.1, C28.1, C29.1, FB1.1, J2.5 (Pin_5), J3.5 (Pin_5), R10.2, R5.1, R7.2, R8.2, R9.2, U4.20 (VCC), U5.1 (VBAT), U5.19 (VDD), U5.32 (VDD), U5.48 (VDD), U5.64 (VDD)
- net GND: now also C18.2, C19.2, C20.2, C21.2, C22.2, C23.2, C24.2, C25.2, C26.2, C27.2, C28.2, C29.2, C30.2, C31.2, C32.1, C33.1, J2.2 (Pin_2), J3.2 (Pin_2), U4.10 (PGND2), U4.18 (GND), U4.3 (PGND1), U4.4 (PGND1), U4.9 (PGND2), U5.12 (VSSA), U5.18 (VSS), U5.63 (VSS)
- new net: C32.2, U5.31 (VCAP_1)
- new net: C33.2, U5.47 (VCAP_2)
- new net: R5.2, U4.19 (STBY)
- new net +3.3VA: C30.1, C31.1, FB1.2, U5.13 (VDDA)
- new net ENC_1A: C22.1, J2.3 (Pin_3), R8.1
- new net ENC_1B: C21.1, J2.4 (Pin_4), R7.1
- new net ENC_2A: C24.1, J3.3 (Pin_3), R10.1
- new net ENC_2B: C23.1, J3.4 (Pin_4), R9.1
- new net J1_MA+: J2.6 (Pin_6), U4.1 (AO1), U4.2 (AO1)
- new net J1_MA-: J2.1 (Pin_1), U4.5 (AO2), U4.6 (AO2)
- new net J2_MB+: J3.6 (Pin_6), U4.11 (BO1), U4.12 (BO1)
- new net J2_MB-: J3.1 (Pin_1), U4.7 (BO2), U4.8 (BO2)
- new net STM32_AIN1: U4.21 (AIN1)
- new net STM32_AIN2: U4.22 (AIN2)
- new net STM32_BIN1: U4.17 (BIN1)
- new net STM32_BIN2: U4.16 (BIN2)
- new net STM32_PWMA: U4.23 (PWMA)
- new net STM32_PWMB: U4.15 (PWMB)
Other:
- note added: "MOTOR DRIVER"
- moved on the sheet: J1

Commit message: update3
Parts:
- added C34, C35: 22pF, Capacitor_SMD:C_0603_1608Metric, symbol Device:C
- added C36, C37: 100nF, Capacitor_SMD:C_0603_1608Metric, symbol Device:C
- added R11, R6: 10kOhm, Resistor_SMD:R_0603_1608Metric, symbol Device:R
- added SW1: SW_Reset, Button_Switch_SMD:SW_SPST_B3U-1000P, symbol Switch:SW_Push
- added SW2: SW_BOOT, Button_Switch_SMD:SW_SPST_B3U-1000P, symbol Switch:SW_Push
- added Y1: 8MHz, Crystal:Crystal_SMD_5032-2Pin_5.0x3.2mm, symbol Device:Crystal
Connections:
- net +3.3V: now also R11.1, SW2.1
- net GND: now also C34.2, C35.2, C36.2, C37.2, R6.2, SW1.2
- net STM32_SWDIO: now reaches U5.46 (PA13)
- net STM32_SWCLK: now reaches U5.49 (PA14)
- net at U5.5 (PH0): now also C34.1, Y1.1
- net at U5.6 (PH1): now also C35.1, Y1.2
- net STM32_BOOT: now reaches U5.60 (BOOT0)
- net STM32_BOOT: now also C36.1, R6.1, SW2.2
- net STM32_RESET: now reaches U5.7 (NRST)
- net STM32_RESET: now also C37.1, R11.2, SW1.1
Other:
- moved on the sheet: C32, C33, U5

Commit message: update4
Parts:
- added C38: 470nF, Capacitor_SMD:C_0603_1608Metric, symbol Device:C
- added C39: 100nF, Capacitor_SMD:C_0603_1608Metric, symbol Device:C
- added J4: ST_Link, Connector_PinHeader_2.54mm:PinHeader_2x04_P2.54mm_Horizontal, symbol Connector_Generic:Conn_02x04_Odd_Even
- added J5, J6: USB_C_Receptacle_USB2.0_16P, Connector_USB:USB_C_Receptacle_HRO_TYPE-C-31-M-12, symbol Connector:USB_C_Receptacle_USB2.0_16P
- added Q1: Q_PMOS_GSD, Package_TO_SOT_SMD:SOT-23, symbol Transistor_FET:Q_PMOS_GSD
- added R12, R13, R21, R22: 5.1kOhm, Resistor_SMD:R_0603_1608Metric, symbol Device:R
- added R14: 10kOhm, Resistor_SMD:R_0603_1608Metric, symbol Device:R
- added R15: 2kOhm, Resistor_SMD:R_0603_1608Metric, symbol Device:R
- added R16: 9kOhm, Resistor_SMD:R_0603_1608Metric, symbol Device:R
- added R17: 1kOhm, Resistor_SMD:R_0603_1608Metric, symbol Device:R
- added R18, R19, R20: 470Ohm, Resistor_SMD:R_0603_1608Metric, symbol Device:R
- added U6: LM358, symbol Amplifier_Operational:LM358
- added U7: CH340E, Package_SO:MSOP-10_3x3mm_P0.5mm, symbol Interface_USB:CH340E
Connections:
- net +12V: no longer C1.1, C2.1, C8.1, U1.2 (VIN), U1.3 (EN)
- net +3.3V: now also C39.1, R14.1, U7.10 (V3), U7.7 (VCC)
- net +5V: now also Q1.3 (D), U6.8 (V+)
- net GND: now also C38.2, C39.2, J4.3 (Pin_3), J4.5 (Pin_5), J4.7 (Pin_7), J4.8 (Pin_8), J5.A1 (GND), J5.A12 (GND), J5.B1 (GND), J5.B12 (GND), J6.A1 (GND), J6.A12 (GND), J6.B1 (GND), J6.B12 (GND), R12.2, R13.2, R15.2, R17.2, R21.1, R22.2, U6.4 (V-), U7.3 (GND)
- net IMU_CS: now also U5.54 (PD2)
- net IMU_INT: now also U5.61 (PB8)
- net IMU_MISO: now also U5.56 (PB4)
- net IMU_MOSI: now also U5.57 (PB5)
- net IMU_SCK: now also U5.55 (PB3)
- net STM32_RESET: now also J4.1 (Pin_1)
- net STM32_SWCLK: now also J4.6 (Pin_6)
- net STM32_SWDIO: now also J4.4 (Pin_4)
- net RX_USB: now reaches U5.14 (PA0)
- net RX_USB: now also R19.2
- net TX_USB: now reaches U5.15 (PA1)
- net TX_USB: now also R20.1
- net USB_DM: now reaches U5.44 (PA11)
- net USB_DM: now also J5.A7 (D-), J5.B7 (D-)
- net USB_DP: now reaches U5.45 (PA12)
- net USB_DP: now also J5.A6 (D+), J5.B6 (D+)
- new net: J6.A5 (CC1), R21.2
- new net: J6.B5 (CC2), R22.1
- new net: R19.1, U7.9 (RXD)
- new net: R20.2, U7.8 (TXD)
- new net: R14.2, R15.1, U6.2 (-)
- new net: R18.1, U6.6 (-), U6.7
- new net: Q1.1 (G), U6.1
- new net: J5.A5 (CC1), R12.1
- new net: J5.B5 (CC2), R13.1
- new net %BAT: C38.1, R18.2
- new net UART_DM: J6.A7 (D-), J6.B7 (D-), U7.2 (UD-)
- new net UART_DP: J6.A6 (D+), J6.B6 (D+), U7.1 (UD+)
- new net VBAT_SNS: R16.2, R17.1, U6.3 (+), U6.5 (+)
- new net VBUS: J4.2 (Pin_2), J5.A4 (VBUS), J5.A9 (VBUS), J5.B4 (VBUS), J5.B9 (VBUS), J6.A4 (VBUS), J6.A9 (VBUS), J6.B4 (VBUS), J6.B9 (VBUS), Q1.2 (S)
- new net VCC: C1.1, C2.1, C8.1, R16.1, U1.2 (VIN), U1.3 (EN)
- no-connect marks 1 -> 10
Other:
- note added: "BATTERY MONITOR"
- note added: "TYPE C TO USART_4 STM32"
- note added: "USB TYPE C"
- note added: "VOLTAGE MCU FILTER"
- moved on the sheet: C1, C10, C11, C12, C13, C14, C15, C16, C17, C18, C19, C2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

Commit message: update5
Parts:
- added D5: LED_RUN, LED_SMD:LED_0603_1608Metric, symbol Device:LED
- added D6: LED_ERR, LED_SMD:LED_0603_1608Metric, symbol Device:LED
- added J7: +12V_BAT, Connector_AMASS:AMASS_XT60PW-M_1x02_P7.20mm_Horizontal, symbol Connector_Generic:Conn_01x02
- added R23, R24: 330 Ohm, Resistor_SMD:R_0603_1608Metric, symbol Device:R
Connections:
- net VCC is gone; now on net +12V_BAT: C1.1, C2.1, C8.1, R16.1, U1.2 (VIN), U1.3 (EN)
- net %BAT: now also U5.21 (PA5)
- net +5V_Pi: now also J1.2 (Pin_2), J1.4 (Pin_4)
- net ENC_1A: now also U5.14 (PA0)
- net ENC_1B: now also U5.15 (PA1)
- net ENC_2A: now also U5.22 (PA6)
- net ENC_2B: now also U5.23 (PA7)
- net GND: now also J1.14 (Pin_14), J1.20 (Pin_20), J1.25 (Pin_25), J1.30 (Pin_30), J1.34 (Pin_34), J1.39 (Pin_39), J1.6 (Pin_6), J1.9 (Pin_9), D5.1 (K), D6.1 (K), J7.2 (Pin_2)
- net RX_USB: now also U5.42 (PA9); no longer U5.14 (PA0)
- net STM32_AIN1: now also U5.8 (PC0)
- net STM32_AIN2: now also U5.9 (PC1)
- net STM32_BIN1: now also U5.10 (PC2)
- net STM32_BIN2: now also U5.11 (PC3)
- net STM32_PWMA: now also U5.39 (PC8)
- net STM32_PWMB: now also U5.40 (PC9)
- net TX_USB: now also U5.43 (PA10); no longer U5.15 (PA1)
- net LED_RUN: now reaches U5.27 (PB1)
- net LED_RUN: now also R23.1
- net LED_ERR: now reaches U5.28 (PB2)
- net LED_ERR: now also R24.1
- net SCL_Pi: now reaches U5.58 (PB6)
- net SCL_Pi: now also J1.5 (Pin_5)
- net SDA_Pi: now reaches U5.59 (PB7)
- net SDA_Pi: now also J1.3 (Pin_3)
- net +12V renamed +12V_BAT
- net +12V_BAT: now also J7.1 (Pin_1)
- new net: D5.2 (A), R23.2
- new net: D6.2 (A), R24.2
Other:
- note added: "LED"
- note added: "MCU CORE & Pi"
- title: (none) -> amr_controller_HAT
- moved on the sheet: C32, C33, C34, C35, C38, C39, J1, J4, J5, J6, Q1, R12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

Commit message: update6
Parts:
- removed C1: 10uF/35V, Capacitor_SMD:C_1206_3216Metric, symbol Device:C
- removed C2: 220nF/50V, Capacitor_SMD:C_0603_1608Metric, symbol Device:C
- removed C3: 1uF/16V, Capacitor_SMD:C_0603_1608Metric, symbol Device:C
- removed C4: 0.1uF/25V, Capacitor_SMD:C_0603_1608Metric, symbol Device:C
- removed C5, C6, C7: 22uF/16V, Capacitor_SMD:C_0805_2012Metric, symbol Device:C
- removed C8: 1000uF/35V, Capacitor_THT:CP_Radial_D10.0mm_P5.00mm, symbol Device:C_US
- removed L1: 6.8uH/4.5A, Inductor_SMD:L_7.3x7.3_H4.5, symbol Device:L
- removed R1: 100kOhm, Resistor_SMD:R_0603_1608Metric, symbol Device:R
- removed R2: 24.9kOhm, Resistor_SMD:R_0603_1608Metric, symbol Device:R
- removed U1: LMR33640ADDA, Package_SO:Texas_HSOP-8-1EP_3.9x4.9mm_P1.27mm_ThermalVias, symbol Regulator_Switching:LMR33640ADDA
- added C40, C47: 10uF, Capacitor_SMD:C_1206_3216Metric, symbol Device:C
- added C41, C44: 0.1uF, Capacitor_SMD:C_0603_1608Metric, symbol Device:C
- added C42: 5pF, Capacitor_SMD:C_0603_1608Metric, symbol Device:C
- added C43: 0.47uF, Capacitor_SMD:C_0603_1608Metric, symbol Device:C
- added C45, C46: 22uF, Capacitor_SMD:C_1206_3216Metric, symbol Device:C
- added C48: 1000uF/35V, Capacitor_THT:CP_Radial_D10.0mm_P5.00mm, symbol Device:C_US
- added L2: 3.3uH, Inductor_SMD:L_7.3x7.3_H4.5, symbol Device:L
- added R25: 374kOhm, Resistor_SMD:R_0603_1608Metric, symbol Device:R
- added R26: 49.9kOhm, Resistor_SMD:R_0603_1608Metric, symbol Device:R
- added R27: 10kOhm, Resistor_SMD:R_0603_1608Metric, symbol Device:R
- added R28: 100kOhm, Resistor_SMD:R_0603_1608Metric, symbol Device:R
- added U9: TPS56528DDA, Package_SO:Texas_HSOP-8-1EP_3.9x4.9mm_P1.27mm_ThermalVias, symbol Regulator_Switching:TPS56528DDA
- F1: value PTC Fuse 3A -> Fuse 2920L500; footprint Fuse:Fuse_1812_4532Metric -> Fuse:Fuse_2920_7451Metric
- J2, J3: footprint Connector_JST:JST_XH_B6B-XH-A_1x06_P2.50mm_Vertical -> Connector_JST:JST_PH_S6B-PH-K_1x06_P2.00mm_Horizontal
Connections:
- net +12V_BAT: now also C40.2, C41.2, C47.2, C48.1, R27.1, U9.8 (VIN)
- net +5V: now also C42.1, C45.1, C46.1, L2.2, R25.2
- net GND: now also C40.1, C41.1, C43.2, C45.2, C46.2, C47.1, C48.2, R26.2, U9.5 (GND), U9.9 (GND)
- new net: C43.1, R28.1, U9.3 (VREG5)
- new net: R27.2, U9.1 (EN)
- new net: C44.2, L2.1, U9.6 (SW)
- new net: C42.2, R25.1, R26.1, U9.2 (VFB)
- new net: R28.2, U9.4 (PG)
- new net: C44.1, U9.7 (VBST)
Other:
- note added: "BUCK CONVERTER Vin: 12V Vout: 5V / 5A"
- note removed: "BUCK CONVERTER Vin: 12V Vout: 5V"
- moved on the sheet: C10, C11, C12, C15, C16, C17, C32, C33, C34, C35, C38, C39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

Commit message: update7
Parts:
- removed D4: TVS_Diode 5.0V, Diode_SMD:D_SMB, symbol Device:D_TVS
- added C1, C2: 2.2uF, Capacitor_SMD:C_0603_1608Metric, symbol Device:C
- added D7: SMAJ5.0A, Diode_SMD:D_SMA, symbol Device:D_Schottky
- added FB2: F120R, Inductor_SMD:L_0603_1608Metric, symbol Device:FerriteBead
- C13: value 22uF/10V -> 100uF; footprint Capacitor_SMD:C_0805_2012Metric -> Capacitor_Tantalum_SMD:CP_EIA-6032-28_Kemet-C
- Q1: value Q_PMOS_GSD -> FDN304P
- U3: footprint BMI323_BOS -> BMI323:BMI323_BOS
Connections:
- net +5V: now also C1.1, FB2.2; no longer Q1.3 (D)
- net +5V_Pi: now also D7.1 (K)
- net GND: now also C1.2, C2.2, D7.2 (A)
- net STM32_BOOT: now also J1.13 (Pin_13)
- net STM32_RESET: now also J1.11 (Pin_11)
- net USART2_TX: now reaches U5.16 (PA2)
- net USART2_TX: now also J1.10 (Pin_10)
- net USART2_RX: now reaches U5.17 (PA3)
- net USART2_RX: now also J1.8 (Pin_8)
- new net: C2.1, FB2.1, Q1.3 (D)

Commit message: update8
Parts:
- removed C13: 100uF, Capacitor_Tantalum_SMD:CP_EIA-6032-28_Kemet-C, symbol Device:C
- removed C14: 100nF/50V, Capacitor_SMD:C_0805_2012Metric, symbol Device:C
- removed D7: SMAJ5.0A, Diode_SMD:D_SMA, symbol Device:D_Schottky
- removed F1: Fuse 2920L500, Fuse:Fuse_2920_7451Metric, symbol Device:Polyfuse_Small
- added J8: USB_A, Connector_USB:USB_A_Molex_67643_Horizontal, symbol Connector:USB_A
Connections:
- net +5V: now also J8.1 (VBUS)
- net GND: now also J8.4 (GND), J8.SH (Shield)
- net +5V_Pi: no longer names the net of J1.2 (Pin_2)
- net +5V_Pi: no longer J1.4 (Pin_4)
- no-connect marks 10 -> 12
Other:
- note removed: "POWER PROTECTION Pi"
- moved on the sheet: C40, C41, C42, C43, C44, C45, C46, C47, C48, J6, J7, L2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
