File: amr_stm32_kicad/amr_stm32_kicad.kicad_sch (KiCad schematic)
At the start: 93 parts, among them J1 Header 2x20, J2 MA, J3 MB, J4 ST_Link, J5 USB_C_Receptacle_USB2.0_16P, J6 USB_C_Receptacle_USB2.0_16P, J7 +12V_BAT, J8 USB_A, Q1 FDN304P, SW1 SW_Reset, SW2 SW_BOOT, U2 SGM2205-3.3, U3 BMI323, U4 TB6612FNG, U5 STM32F405RGTx, U6 LM358, U7 CH340E, U9 TPS56528DDA, Y1 8MHz

Commit message: update8
Parts:
- removed Y1: 8MHz, Crystal:Crystal_SMD_5032-2Pin_5.0x3.2mm, symbol Device:Crystal
- added Y2: 8MHz, Crystal:Crystal_SMD_5032-4Pin_5.0x3.2mm, symbol Device:Crystal_GND24
- C32, C33: footprint Capacitor_SMD:C_0603_1608Metric -> Capacitor_SMD:C_0805_2012Metric
- J5: value USB_C_Receptacle_USB2.0_16P -> USB_FS_Interface
- J6: value USB_C_Receptacle_USB2.0_16P -> USB_UART
Connections:
- net GND: now also J4.1 (Pin_1), J4.2 (Pin_2), J5.SH (SHIELD), J6.SH (SHIELD), Y2.2 (G), Y2.4 (G); no longer J4.7 (Pin_7), J4.8 (Pin_8)
- net STM32_RESET: now also J4.7 (Pin_7); no longer J4.1 (Pin_1)
- net STM32_SWCLK: now also J4.4 (Pin_4); no longer J4.6 (Pin_6)
- net STM32_SWDIO: now also J4.6 (Pin_6); no longer J4.4 (Pin_4)
- net VBUS: now also J4.8 (Pin_8); no longer J4.2 (Pin_2)
- net PC13: now reaches U5.2 (PC13)
- net PA4: now reaches U5.20 (PA4)
- net PC4: now reaches U5.24 (PC4)
- net PC5: now reaches U5.25 (PC5)
- net PB0: now reaches U5.26 (PB0)
- net PB10: now reaches U5.29 (PB10)
- net PC14: now reaches U5.3 (PC14)
- net PB11: now reaches U5.30 (PB11)
- net PB12: now reaches U5.33 (PB12)
- net PB13: now reaches U5.34 (PB13)
- net PB14: now reaches U5.35 (PB14)
- net PB15: now reaches U5.36 (PB15)
- net PC6: now reaches U5.37 (PC6)
- net PC7: now reaches U5.38 (PC7)
- net PC15: now reaches U5.4 (PC15)
- net PA8: now reaches U5.41 (PA8)
- net at C34.1, U5.5 (PH0): now also Y2.3
- net PA15: now reaches U5.50 (PA15)
- net PC10: now reaches U5.51 (PC10)
- net PC11: now reaches U5.52 (PC11)
- net PC12: now reaches U5.53 (PC12)
- net at C35.1, U5.6 (PH1): now also Y2.1
- net PB9: now reaches U5.62 (PB9)
- no-connect marks 12 -> 10
Other:
- moved on the sheet: C37, R11, SW1

Commit message: update10
Parts:
- added J10: VCC, Connector_PinSocket_2.54mm:PinSocket_1x06_P2.54mm_Vertical, symbol Connector_Generic:Conn_01x06
- added J9: UART, Connector_PinSocket_2.54mm:PinSocket_1x06_P2.54mm_Vertical, symbol Connector_Generic:Conn_01x06
- D1: value D_Schottky 5A/40V -> D_Schottky 1A/40V; footprint Diode_SMD:D_SMC -> Diode_SMD:D_SOD-123
- J2: value MA -> Motor_Left
- J3: value MB -> Motor_right
- J8: value USB_A -> USB_A_Pi
Connections:
- net +3.3V: now also J10.3 (Pin_3), J10.4 (Pin_4)
- net +5V: now also J10.5 (Pin_5), J10.6 (Pin_6), J9.2 (Pin_2)
- net GND: now also J10.1 (Pin_1), J10.2 (Pin_2), J9.3 (Pin_3)
- net PC10 renamed USART3_TX
- net USART3_TX: now also J9.5 (Pin_5)
- net PC11 renamed USART3_RX
- net USART3_RX: now also J9.4 (Pin_4)
Other:
- moved on the sheet: J4

Commit message: update11
Parts:
- added C49: 100nF/50V, Capacitor_SMD:C_0805_2012Metric, symbol Device:C
Connections:
- net PB10 is gone; now on net STM32_PWMA: U5.29 (PB10)
- net PB11 is gone; now on net STM32_PWMB: U5.30 (PB11)
- net +12V_BAT: now also C49.1
- net GND: now also C49.2
- net STM32_PWMA: no longer U5.39 (PC8)
- net STM32_PWMB: no longer U5.40 (PC9)
- new net PC8: U5.39 (PC8)
- new net PC9: U5.40 (PC9)
Changed lines of the file:
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@@
 	)
 	(junction
-		(at 100.33 45.72)
-		(diameter 0)
-		(color 0 0 0 0)
-	)
-	(junction
-		(at 382.27 119.38)
+		(at 425.45 38.1)
 		(diameter 0)
 		(color 0 0 0 0)
 	)
 	(junction
-		(at 281.94 26.67)
+		(at 100.33 45.72)
 		(diameter 0)
 		(color 0 0 0 0)
 	)
 	(junction
-		(at 78.74 35.56)
+		(at 382.27 119.38)
 		(diameter 0)
 		(color 0 0 0 0)
 	)
 	(junction
-		(at 78.74 45.72)
+		(at 281.94 26.67)
 		(diameter 0)
 		(color 0 0 0 0)
@@
 	)
 	(junction
+		(at 425.45 29.21)
+		(diameter 0)
+		(color 0 0 0 0)
+	)
+	(junction
 		(at 86.36 177.8)
 		(diameter 0)
@@
 	)
 	(junction
+		(at 78.74 35.56)
+		(diameter 0)
+		(color 0 0 0 0)
+	)
+	(junction
+		(at 78.74 45.72)
+		(diameter 0)
+		(color 0 0 0 0)
+	)
+	(junction
 		(at 293.37 35.56)
 		(diameter 0)
@@
 	(wire
 		(pts
-			(xy 419.1 38.1) (xy 431.8 38.1)
+			(xy 419.1 38.1) (xy 425.45 38.1)
 		)
 		(stroke
@@
 	(wire
 		(pts
+			(xy 425.45 30.48) (xy 425.45 29.21)
+		)
+		(stroke
+			(width 0)
+			(type default)
+		)
+	)
+	(wire
+		(pts
 			(xy 358.14 193.04) (xy 368.3 193.04)
 		)
@@
 	(wire
 		(pts
+			(xy 425.45 29.21) (xy 431.8 29.21)
+		)
+		(stroke
+			(width 0)
+			(type default)
+		)
+	)
+	(wire
+		(pts
 			(xy 144.78 195.58) (xy 148.59 195.58)
 		)
@@
 	(wire
 		(pts
+			(xy 425.45 38.1) (xy 431.8 38.1)
+		)
+		(stroke
+			(width 0)
+			(type default)
+		)
+	)
+	(wire
+		(pts
 			(xy 429.26 251.46) (xy 434.34 251.46)
 		)
@@
 	(wire
 		(pts
-			(xy 419.1 29.21) (xy 431.8 29.21)
+			(xy 419.1 29.21) (xy 425.45 29.21)
 		)
 		(stroke
@@
 		)
 	)
-	(label "PB11"
+	(label "STM32_PWMB"
 		(at 368.3 261.62 0)
 		(effects
@@
 		)
 	)
-	(label "PB10"
+	(label "STM32_PWMA"
 		(at 368.3 259.08 0)
 		(effects
@@
 		)
 	)
-	(label "STM32_PWMB"
+	(label "PC9"
 		(at 300.99 236.22 0)
 		(effects
@@
 		)
 	)
-	(label "STM32_PWMA"
+	(label "PC8"
 		(at 300.99 233.68 0)
 		(effects
@@
 		)
 	)
+	(symbol
+		(lib_id "Device:C")
+		(at 425.45 34.29 0)
+		(unit 1)
+		(body_style 1)
+		(exclude_from_sim no)
+		(in_bom yes)
+		(on_board yes)
+		(in_pos_files yes)
+		(dnp no)
+		(property "Reference" "C49"
+			(at 429.26 33.0199 0)
+			(show_name no)
+			(do_not_autoplace no)
+			(effects
+				(font
+					(size 1.27 1.27)
+				)
+				(justify left)
+			)
+		)
+		(property "Value" "100nF/50V"
+			(at 417.83 26.67 0)
+			(show_name no)
+			(do_not_autoplace no)
+			(effects
+				(font
+					(size 1.27 1.27)
+				)
+				(justify left)
+			)
+		)
+		(property "Footprint" "Capacitor_SMD:C_0805_2012Metric"
+			(at 426.4152 38.1 0)
+			(hide yes)
+			(show_name no)
+			(do_not_autoplace no)
+			(effects
+				(font
+					(size 1.27 1.27)
+				)
+			)
+		)
+		(property "Datasheet" ""
+			(at 425.45 34.29 0)
+			(hide yes)
+			(show_name no)
+			(do_not_autoplace no)
+			(effects
+				(font
+					(size 1.27 1.27)
+				)
+			)
+		)
+		(property "Description" "Unpolarized capacitor"
+			(at 425.45 34.29 0)
+			(hide yes)
+			(show_name no)
+			(do_not_autoplace no)
+			(effects
+				(font
+					(size 1.27 1.27)
+				)
+			)
+		)
+		(pin "1"
+		)
+		(pin "2"
+		)
+		(instances
+			(project "amr_stm32_kicad"
+				(path "/cf072b7b-77da-4611-a2b1-45164595d9a3"
+					(reference "C49")
+					(unit 1)
+				)
+			)
+		)
+	)

Commit message: update14
Parts:
- U3: footprint BMI323:BMI323_BOS -> BMI323:BMI323_BOS-L
Changed lines of the file:
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@@
 			)
 		)
-		(property "Footprint" "BMI323:BMI323_BOS"
+		(property "Footprint" "BMI323:BMI323_BOS-L"
 			(at 209.55 134.62 0)
 			(hide yes)

Commit message: update19
Connections:
- net PC4 is gone; now on net LED_RUN: U5.24 (PC4)
- net PC5 is gone; now on net LED_ERR: U5.25 (PC5)
- net LED_ERR: no longer U5.28 (PB2)
- net LED_RUN: no longer U5.27 (PB1)
- new net PB1: U5.27 (PB1)
- new net PB2: U5.28 (PB2)
Changed lines of the file:
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@@
 		)
 	)
-	(label "LED_ERR"
+	(label "PB2"
 		(at 368.3 238.76 0)
 		(effects
@@
 		)
 	)
-	(label "PC5"
+	(label "LED_ERR"
 		(at 300.99 226.06 0)
 		(effects
@@
 		)
 	)
-	(label "PC4"
+	(label "LED_RUN"
 		(at 300.99 223.52 0)
 		(effects
@@
 		)
 	)
-	(label "LED_RUN"
+	(label "PB1"
 		(at 368.3 236.22 0)
 		(effects

Commit message: update20
Parts:
- added D7: LED_ERR, LED_SMD:LED_0603_1608Metric, symbol Device:LED
- added R29: 330 Ohm, Resistor_SMD:R_0603_1608Metric, symbol Device:R
Connections:
- net PC12 is gone; now on net IMU_INT: U5.53 (PC12)
- net GND: now also D7.1 (K)
- net IMU_INT: no longer U5.61 (PB8)
- net LED_ERR renamed LED_2
- net LED_RUN renamed LED_1
- net PB0 renamed LED_3
- net LED_3: now also R29.1
- new net: D7.2 (A), R29.2
- new net PB8: U5.61 (PB8)
Other:
- moved on the sheet: D5, D6, R23, R24

Commit message: update23
Connections:
- net STM32_BOOT: no longer J1.13 (Pin_13)
- net STM32_RESET: no longer J1.11 (Pin_11)
Changed lines of the file:
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@@
 	(wire
 		(pts
-			(xy 424.18 198.12) (xy 439.42 198.12)
-		)
-		(stroke
-			(width 0)
-			(type default)
-		)
-	)
-	(wire
-		(pts
 			(xy 358.14 259.08) (xy 368.3 259.08)
 		)
@@
 	(wire
 		(pts
-			(xy 424.18 200.66) (xy 439.42 200.66)
-		)
-		(stroke
-			(width 0)
-			(type default)
-		)
-	)
-	(wire
-		(pts
 			(xy 209.55 54.61) (xy 209.55 59.69)
 		)
@@
 		)
 	)
-	(label "STM32_RESET"
-		(at 424.18 198.12 0)
-		(effects
-			(font
-				(size 1.27 1.27)
-			)
-			(justify left bottom)
-		)
-	)
 	(label "UART_DP"
 		(at 120.65 283.21 0)
@@
 		(effects
 			(font
-				(size 1.27 1.27)
-			)
-			(justify left bottom)
-		)
-	)
-	(label "STM32_BOOT"
-		(at 424.18 200.66 0)
-		(effects
-			(font

Commit message: update28
Connections:
- net +5V: now also L2.1; no longer L2.2
- net at C44.2, U9.6 (SW): now also L2.2; no longer L2.1
Other:
- moved on the sheet: L2
Changed lines of the file:
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@@
 	(symbol
 		(lib_id "Device:L")
-		(at 189.23 54.61 90)
+		(at 189.23 54.61 270)
+		(mirror x)
 		(unit 1)
 		(body_style 1)
