File: amr_stm32_kicad/amr_stm32_kicad.kicad_sch (KiCad schematic)
At the start: 98 parts, among them J1 Header 2x20, J10 VCC, J2 Motor_Left, J3 Motor_right, J4 ST_Link, J5 USB_FS_Interface, J6 USB_UART, J7 +12V_BAT, J8 USB_A_Pi, J9 UART, Q1 FDN304P, SW1 SW_Reset, SW2 SW_BOOT, U2 SGM2205-3.3, U3 BMI323, U4 TB6612FNG, U5 STM32F405RGTx, U6 LM358, U7 CH340E, U9 TPS56528DDA, Y2 8MHz

Commit message: update29
Parts:
- R3: value 1kOhm -> 300Ohm
- U2: value SGM2205-3.3 -> AP2112K-3.3
Changed lines of the file:
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@@
 		(dnp no)
 		(property "Reference" "C49"
-			(at 429.26 33.0199 0)
+			(at 424.942 40.894 0)
 			(show_name no)
 			(do_not_autoplace no)
@@
 		)
 		(property "Value" "100nF/50V"
-			(at 417.83 26.67 0)
+			(at 419.1 26.416 0)
 			(show_name no)
 			(do_not_autoplace no)
@@
 		)
 		(property "Value" "10uF"
-			(at 66.294 42.672 0)
+			(at 80.264 43.18 0)
 			(show_name no)
 			(do_not_autoplace no)
@@
 			)
 		)
-		(property "Value" "SGM2205-3.3"
+		(property "Value" "AP2112K-3.3"
 			(at 68.58 115.57 0)
 			(show_name no)
@@
 			)
 		)
-		(property "Value" "1kOhm"
+		(property "Value" "300Ohm"
 			(at 96.52 115.57 90)
 			(show_name no)
@@
 		(dnp no)
 		(property "Reference" "C19"
-			(at 422.91 33.0199 0)
+			(at 416.052 41.148 0)
 			(show_name no)
 			(do_not_autoplace no)
@@
 		)
 		(property "Value" "100nF/50V"
-			(at 411.48 26.67 0)
+			(at 403.86 25.908 0)
 			(show_name no)
 			(do_not_autoplace no)

Commit message: update30
Parts:
- removed U2: AP2112K-3.3, Package_TO_SOT_SMD:SOT-23-5, symbol Regulator_Linear:AP2112K-3.3
- added U1: SGM2205_3.3, Package_TO_SOT_SMD:SOT-223-3_TabPin2, symbol Regulator_Linear:AP2204R-3.3
Connections:
- net +12V_BAT: now also J7.2 (Pin_2); no longer J7.1 (Pin_1)
- net +3.3V: now also U1.3 (VOUT)
- net GND: now also J7.1 (Pin_1), U1.2 (GND); no longer J7.2 (Pin_2)
- net at C10.1, C9.1, D1.1 (K)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: now also U1.1 (VIN)
Changed lines of the file:
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@@
 	)
 	(junction
-		(at 55.88 119.38)
-		(diameter 0)
-		(color 0 0 0 0)
-	)
-	(junction
 		(at 293.37 26.67)
 		(diameter 0)
@@
 	)
 	(junction
+		(at 67.31 133.35)
+		(diameter 0)
+		(color 0 0 0 0)
+	)
+	(junction
 		(at 393.7 85.09)
 		(diameter 0)
@@
 	)
 	(junction
-		(at 68.58 133.35)
-		(diameter 0)
-		(color 0 0 0 0)
-	)
-	(junction
 		(at 171.45 63.5)
 		(diameter 0)
@@
 	(wire
 		(pts
-			(xy 68.58 133.35) (xy 68.58 129.54)
-		)
-		(stroke
-			(width 0)
-			(type default)
-		)
-	)
-	(wire
-		(pts
 			(xy 458.47 48.26) (xy 454.66 48.26)
 		)
@@
 	(wire
 		(pts
-			(xy 55.88 121.92) (xy 60.96 121.92)
-		)
-		(stroke
-			(width 0)
-			(type default)
-		)
-	)
-	(wire
-		(pts
 			(xy 167.64 288.29) (xy 167.64 294.64)
 		)
@@
 	(wire
 		(pts
-			(xy 222.25 260.35) (xy 222.25 273.05)
+			(xy 67.31 127) (xy 67.31 133.35)
 		)
 		(stroke
@@
 	(wire
 		(pts
-			(xy 49.53 109.22) (xy 49.53 119.38)
+			(xy 222.25 260.35) (xy 222.25 273.05)
 		)
 		(stroke
@@
 	(wire
 		(pts
-			(xy 429.26 254) (xy 434.34 254)
+			(xy 49.53 109.22) (xy 49.53 119.38)
 		)
 		(stroke
@@
 	(wire
 		(pts
-			(xy 458.47 279.4) (xy 463.55 279.4)
+			(xy 429.26 254) (xy 434.34 254)
 		)
 		(stroke
@@
 	(wire
 		(pts
-			(xy 76.2 119.38) (xy 81.28 119.38)
+			(xy 458.47 279.4) (xy 463.55 279.4)
 		)
 		(stroke
@@
 	(wire
 		(pts
+			(xy 74.93 119.38) (xy 81.28 119.38)
+		)
+		(stroke
+			(width 0)
+			(type default)
+		)
+	)
+	(wire
+		(pts
 			(xy 293.37 55.88) (xy 293.37 57.15)
 		)
@@
 	(wire
 		(pts
-			(xy 55.88 119.38) (xy 60.96 119.38)
-		)
-		(stroke
-			(width 0)
-			(type default)
-		)
-	)
-	(wire
-		(pts
 			(xy 426.72 281.94) (xy 431.8 281.94)
 		)
@@
 	(wire
 		(pts
+			(xy 67.31 133.35) (xy 81.28 133.35)
+		)
+		(stroke
+			(width 0)
+			(type default)
+		)
+	)
+	(wire
+		(pts
 			(xy 293.37 66.04) (xy 300.99 66.04)
 		)
@@
 	(wire
 		(pts
-			(xy 68.58 133.35) (xy 81.28 133.35)
+			(xy 60.96 133.35) (xy 67.31 133.35)
 		)
 		(stroke
@@
 	(wire
 		(pts
-			(xy 55.88 119.38) (xy 55.88 121.92)
-		)
-		(stroke
-			(width 0)
-			(type default)
-		)
-	)
-	(wire
-		(pts
 			(xy 382.27 85.09) (xy 393.7 85.09)
 		)
@@
 	(wire
 		(pts
-			(xy 60.96 133.35) (xy 68.58 133.35)
-		)
-		(stroke
-			(width 0)
-			(type default)
-		)
-	)
-	(wire
-		(pts
 			(xy 471.17 64.77) (xy 471.17 68.58)
 		)
@@
 	(wire
 		(pts
-			(xy 49.53 119.38) (xy 55.88 119.38)
+			(xy 49.53 119.38) (xy 59.69 119.38)
 		)
 		(stroke
@@
 		)
 	)
-	(label "+12V_BAT"
+	(label "GND"
 		(at 49.53 77.47 0)
 		(effects
@@
 		)
 	)
-	(label "GND"
+	(label "+12V_BAT"
 		(at 49.53 74.93 0)
 		(effects
@@
 	)
 	(symbol
+		(lib_id "Regulator_Linear:AP2204R-3.3")
+		(at 67.31 119.38 0)
+		(unit 1)
+		(body_style 1)
+		(exclude_from_sim no)
+		(in_bom yes)
+		(on_board yes)
+		(in_pos_files yes)
+		(dnp no)
+		(fields_autoplaced yes)
+		(property "Reference" "U1"
+			(at 67.31 113.03 0)
+			(show_name no)
+			(do_not_autoplace no)
+			(effects
+				(font
+					(size 1.27 1.27)
+				)
+			)
+		)
+		(property "Value" "SGM2205_3.3"
+			(at 67.31 115.57 0)
+			(show_name no)
+			(do_not_autoplace no)
+			(effects
+				(font
+					(size 1.27 1.27)
+				)
+			)
+		)
+		(property "Footprint" "Package_TO_SOT_SMD:SOT-223-3_TabPin2"
+			(at 67.31 113.665 0)
+			(hide yes)
+			(show_name no)
+			(do_not_autoplace no)
+			(effects
+				(font
+					(size 1.27 1.27)
+				)
+			)
+		)
+		(property "Datasheet" "https://www.diodes.com/assets/Datasheets/products_inactive_data/AP2204.pdf"
+			(at 67.31 119.38 0)
+			(hide yes)
+			(show_name no)
+			(do_not_autoplace no)
+			(effects
+				(font
+					(size 1.27 1.27)
+				)
+			)
+		)
+		(property "Description" "150mA low dropout linear regulator, wide input voltage range, 3.3V fixed positive output, SOT-89-3 package"
+			(at 67.31 119.38 0)
+			(hide yes)
+			(show_name no)
+			(do_not_autoplace no)
+			(effects
+				(font
+					(size 1.27 1.27)
+				)
+			)
+		)
+		(pin "2"
+		)
+		(pin "1"
+		)
+		(pin "3"
+		)
+		(instances
+			(project "amr_stm32_kicad"
+				(path "/cf072b7b-77da-4611-a2b1-45164595d9a3"
+					(reference "U1")
+					(unit 1)
+				)
+			)
+		)
+	)
+	(symbol
 		(lib_id "Device:R")
 		(at 83.82 52.07 90)
@@
 	)
 	(symbol
-		(lib_id "Regulator_Linear:AP2112K-3.3")
-		(at 68.58 121.92 0)
-		(unit 1)
-		(body_style 1)
-		(exclude_from_sim no)
-		(in_bom yes)
-		(on_board yes)
-		(in_pos_files yes)
-		(dnp no)
-		(fields_autoplaced yes)
-		(property "Reference" "U2"
-			(at 68.58 113.03 0)
-			(show_name no)
-			(do_not_autoplace no)
-			(effects
-				(font
-					(size 1.27 1.27)
-				)
-			)
-		)
-		(property "Value" "AP2112K-3.3"
-			(at 68.58 115.57 0)
-			(show_name no)
-			(do_not_autoplace no)
-			(effects
-				(font
-					(size 1.27 1.27)
-				)
-			)
-		)
-		(property "Footprint" "Package_TO_SOT_SMD:SOT-23-5"
-			(at 68.58 113.665 0)
-			(hide yes)
-			(show_name no)
-			(do_not_autoplace no)
-			(effects
-				(font
-					(size 1.27 1.27)
-				)
-			)
-		)
-		(property "Datasheet" "https://www.diodes.com/assets/Datasheets/AP2112.pdf"
-			(at 68.58 119.38 0)
-			(hide yes)
-			(show_name no)
-			(do_not_autoplace no)
-			(effects
-				(font
-					(size 1.27 1.27)
-				)
-			)
-		)
-		(property "Description" "600mA low dropout linear regulator, with enable pin, 3.8V-6V input voltage range, 3.3V fixed positive output, SOT-23-5"
-			(at 68.58 121.92 0)
-			(hide yes)
-			(show_name no)
-			(do_not_autoplace no)
-			(effects
-				(font
-					(size 1.27 1.27)
-				)
-			)
-		)
-		(pin "3"
-		)
-		(pin "1"
-		)
-		(pin "2"
-		)
-		(pin "5"
-		)
-		(pin "4"
-		)
-		(instances
-			(project "amr_stm32_kicad"
-				(path "/cf072b7b-77da-4611-a2b1-45164595d9a3"
-					(reference "U2")
-					(unit 1)
-				)
-			)
-		)
-	)
-	(symbol
 		(lib_id "Device:C")
 		(at 382.27 127 0)
@@
 		(in_pos_files yes)
 		(dnp no)
-		(fields_autoplaced yes)
 		(property "Reference" "D3"
 			(at 106.68 126.0474 90)

Commit message: update_ide
Parts:
- U6: value LM358 -> LMV358; footprint (none) -> Package_SO:SOIC-8_3.9x4.9mm_P1.27mm
- U6: value LM358 -> LMV358
Changed lines of the file:
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@@
 			)
 		)
-		(property "Value" "LM358"
+		(property "Value" "LMV358"
 			(at 54.61 274.32 0)
 			(show_name no)
@@
 			)
 		)
-		(property "Footprint" ""
+		(property "Footprint" "Package_SO:SOIC-8_3.9x4.9mm_P1.27mm"
 			(at 54.61 281.94 0)
 			(hide yes)
@@
 			)
 		)
-		(property "Value" "LM358"
+		(property "Value" "LMV358"
 			(at 113.03 167.64 0)
 			(show_name no)
@@
 			)
 		)
-		(property "Value" "LM358"
+		(property "Value" "LMV358"
 			(at 53.34 170.18 90)
 			(show_name no)
@@
 			)
 		)
-		(property "Footprint" ""
+		(property "Footprint" "Package_SO:SOIC-8_3.9x4.9mm_P1.27mm"
 			(at 53.34 170.18 0)
 			(hide yes)

Commit message: update9_10
Parts:
- removed Q1: FDN304P, Package_TO_SOT_SMD:SOT-23, symbol Transistor_FET:Q_PMOS_GSD
- removed R14: 10kOhm, Resistor_SMD:R_0603_1608Metric, symbol Device:R
- removed R15: 2kOhm, Resistor_SMD:R_0603_1608Metric, symbol Device:R
- removed unit 1 of U6
- added D4: D_Schottky 1A/40V, Diode_SMD:D_SOD-123, symbol Device:D_Schottky
Connections:
- net VBUS: now also D4.2 (A)
- net at C2.1, FB2.1: now also D4.1 (K)
Other:
- moved on the sheet: C1, C2, FB2, U6C
